File: hardware/hardware.sch (KiCad schematic (older format))
At the start: 47 parts, among them J1 USB_B_Micro, J2 Conn_Coaxial, J3 Breakout, Q1 FS8205, U1 DW01+G, U2 USBLC6-2, U3 MAX2871ETJ+, U4 LM317A, U5 TP4056, U6 PIC18F45K50_QFP, X1 SG-310SCF

Commit message: MAX2871 decoupling.
Parts:
- added C7, C? (x5): 100pf, Capacitor_SMD:C_0603_1608Metric_Pad1.05x0.95mm_HandSolder, symbol Device:C
- added C8, C? (x5): 10nF, Capacitor_SMD:C_0603_1608Metric_Pad1.05x0.95mm_HandSolder, symbol Device:C
- added R3: 4.7k, Resistor_SMD:R_0603_1608Metric_Pad1.05x0.95mm_HandSolder, symbol Device:R
- renumbered C4 to C10, C5 to C11, C6 to C12, C7 to C13, C8 to C14, C9 to C15, C10 to C16, C11 to C17, C12 to C18, C13 to C19, C14 to C20, C15 to C21, C16 to C22, C17 to C23, C18 to C24, C19 to C25, C1 to C3, C2 to C6, C3 to C9, R9 to R10, R10 to R11, R11 to R12, R3 to R4, R4 to R5, R5 to R6, R6 to R7, R7 to R8, R8 to R9
Connections:
- net GND: now also C7.2, C8.2, C?.1, C?.1, C?.1, C?.1, C?.1, C?.1, C?.2, C?.2, C?.2, C?.2, R3.2
- net VDD: now also U3.10 (VCC_PLL), U3.16 (VCC_RF), U3.17 (VCC_VCO), U3.28 (VCC_DIG), U3.32 (VCC_SD), U3.6 (VCC_CP), C7.1, C8.1, C?.1, C?.1, C?.1, C?.1, C?.2, C?.2, C?.2, C?.2, C?.2, C?.2
- net at U3.22 (RSET): now also R3.1
Other:
- note added: "Decoupling"
- moved on the sheet: C10, C11, C12, J2, U3
