File: hardware/hardware.sch (KiCad schematic (older format))
At the start: 68 parts, among them J1 RF A-N, J2 RF A-P, J3 RF B-N, J4 RF B-P, J5 Breakout, J6 USB_B_Micro, U1 MAX2871ETJ+, U2 USBLC6-2, U3 LM317A, X1 SG-310SCF

Commit message: Added TQFN-32 model.
Parts:
- removed C28, C29: 0.1μF, Capacitor_SMD:C_0805_2012Metric_Pad1.15x1.40mm_HandSolder, symbol Device:C
- removed C30: 10μF, Capacitor_SMD:C_0805_2012Metric_Pad1.15x1.40mm_HandSolder, symbol Device:CP
- removed C31: 1μF, Capacitor_SMD:C_0805_2012Metric_Pad1.15x1.40mm_HandSolder, symbol Device:C
- removed D1: M7, Diode_SMD:D_MiniMELF_Handsoldering, symbol Device:D
- removed J5: Breakout, Connector_PinHeader_2.54mm:PinHeader_1x06_P2.54mm_Vertical, symbol Connector_Generic:Conn_01x06
- removed J6: USB_B_Micro, Connector_USB:USB_Micro-B_Molex_47346-0001, symbol Connector:USB_B_Micro
- removed R24: 1k, Resistor_SMD:R_1206_3216Metric_Pad1.42x1.75mm_HandSolder, symbol Device:R
- removed R25: 1.5k, Resistor_SMD:R_1206_3216Metric_Pad1.42x1.75mm_HandSolder, symbol Device:R
- removed U2: USBLC6-2, Package_TO_SOT_SMD:SOT-23-6_Handsoldering, symbol Missing:USBLC6-2
- removed U3: LM317A, Package_TO_SOT_SMD:TO-252-2, symbol Regulator_Linear:LM317_3PinPackage
- removed X1: SG-310SCF, Crystal:Crystal_SMD_3225-4Pin_3.2x2.5mm_HandSoldering, symbol Missing:SG-310SCF
- added J5: Breakout, Connector_PinHeader_2.54mm:PinHeader_1x08_P2.54mm_Vertical, symbol Connector_Generic:Conn_01x08
- added X1: CXO_DIP14, Oscillator:Oscillator_DIP-14, symbol Oscillator:CXO_DIP14
- J1, J2, J3, J4: footprint Connector_Coaxial:SMA_Amphenol_132291_Vertical -> Connector_Coaxial:SMA_Amphenol_901-144_Vertical
- U1: footprint MAX:MAX2871 -> MAX:MAX2871ETJ+
Connections:
- net labels removed: BP_VDD, USB_D+, USB_D-, USB_VBUS
- wire segments 259 -> 218
- no-connect marks 2 -> 0
Other:
- note removed: "3.3V Voltage Regulator \w Improved Ripple Rejection"
- note removed: "USB Connection & ESD Protection"

Commit message: Fixed minor issue with RF Output.
Parts:
- removed X1: CXO_DIP14, Oscillator:Oscillator_DIP-14, symbol Oscillator:CXO_DIP14
- added X?: SG-310SCF, Crystal:Crystal_SMD_3225-4Pin_3.2x2.5mm_HandSoldering, symbol MAX:SG-310SCF
- C1, C10, C11, C12, C13, C14, C15, C16, C17, C18, C19, C2, C20, C21, C22, C23, C24, C25, C26, C27, C3, C4, C5, C6, C7, C8, C9: footprint Capacitor_SMD:C_0805_2012Metric_Pad1.15x1.40mm_HandSolder -> Capacitor_SMD:C_0603_1608Metric_Pad1.05x0.95mm_HandSolder
- JP1: footprint Connector_PinHeader_2.54mm:PinHeader_1x02_P2.54mm_Vertical -> Connector_PinHeader_1.27mm:PinHeader_1x02_P1.27mm_Vertical
- R1, R10, R11, R12, R13, R14, R15, R16, R17, R18, R19, R2, R20, R21, R22, R23, R3, R4, R5, R6, R7, R8, R9: footprint Resistor_SMD:R_1206_3216Metric_Pad1.42x1.75mm_HandSolder -> Resistor_SMD:R_0603_1608Metric_Pad1.05x0.95mm_HandSolder
- U1: symbol Missing:MAX2871ETJ+ -> MAX:MAX2871ETJ+
Connections:
- net GND: now also J1.2 (Ext), J2.2 (Ext), J3.2 (Ext), J4.2 (Ext), R12.2, R13.2, R15.2, R16.2, R2.2, R3.2, R5.2, R6.2, X?.2 (GND)
- net VCC_CP: now also X?.4 (VCC)
- net LD: now reaches U1.25 (LD)
Other:
- note added: "VCO"
- moved on the sheet: C1, C10, C11, C12, C13, C14, C15, C16, C17, C18, C19, C2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
