File: hardware-cvco/hardware.sch (KiCad schematic (older format))
At the start: 126 parts, among them J1 SMA, J2 SMA, J3 SMA, J4 SMA, J6 SMA, J7 SMA, J8 SMA, U1 L78L05_SOT89, U11 L78L12_SOT89, U12 L78L10_SOT89, U13 NLB-310-T1, U14 NLB-310-T1, U16 L78L10_SOT89, U17 NLB-310-T1, U2 L78L05_SOT89, U3 NLB-310-T1, U4 NLB-310-T1, U6 L78L12_SOT89, U7 L78L08_SOT89, U8 NLB-310-T1, U9 NLB-310-T1, Y1 CVCO55CW-0100-0200, Y2 CV55BE1600-3200, Y3 CVCO55CW-0200-0500, Y4 CVCO55CC-3180-3710, Y5 CV55CW500-1000, Y6 CVCO55CW-3500-4500, Y7 CVCO55CW-1000-2000

Commit message: Pover supply for CVCO variant.
Parts:
- added C64: 0.1μF, Capacitor_SMD:C_0805_2012Metric_Pad1.15x1.40mm_HandSolder, symbol Device:C
- added C65: 1μF, Capacitor_SMD:C_0805_2012Metric_Pad1.15x1.40mm_HandSolder, symbol Device:C
- added C66: 10μF, Capacitor_SMD:C_0805_2012Metric_Pad1.15x1.40mm_HandSolder, symbol Device:C
- added D8: 3V, Package_TO_SOT_SMD:SOT-23, symbol Device:D_Zener
- added D9: 1N4002, Diode_SMD:D_SMA_Handsoldering, symbol Device:D
- added J8: DC, Connector_BarrelJack:BarrelJack_Wuerth_6941xx301002, symbol Connector_Generic:Conn_01x02
- added Q1: AOD403, Package_TO_SOT_SMD:TO-252-2, symbol Device:Q_PMOS_GDS
- added R22: 4.7k, Resistor_SMD:R_0805_2012Metric_Pad1.15x1.40mm_HandSolder, symbol Device:R
- added R23: 100k, Resistor_SMD:R_0805_2012Metric_Pad1.15x1.40mm_HandSolder, symbol Device:R
- added R24: 10k, Resistor_SMD:R_0805_2012Metric_Pad1.15x1.40mm_HandSolder, symbol Device:R
- added U15: LM317DCYR, Package_TO_SOT_SMD:SOT-223-3_TabPin2, symbol Regulator_Linear:LM317_3PinPackage
- added U16: MCP73871-2AA, Package_DFN_QFN:QFN-20-1EP_4x4mm_P0.5mm_EP2.5x2.5mm, symbol Battery_Management:MCP73871-2AA
- renumbered C7 to C1, C9 to C10, C23 to C11, C27 to C12, C41 to C13, C45 to C14, C57 to C15, C59 to C16, C15 to C17, C17 to C18, C33 to C19, C13 to C2, C35 to C20, C51 to C21, C53 to C22, C62 to C23, C63 to C24, C11 to C25, C29 to C26, C47 to C27, C60 to C28, C1 to C29, C25 to C3, C3 to C30, C19 to C31, C21 to C32, C37 to C33, C39 to C34, C55 to C35, C56 to C36, C44 to C37, C50 to C38, C8 to C39, C31 to C4, C14 to C40, C26 to C41, C32 to C42, C42 to C43, C46 to C44, C6 to C45, C10 to C46, C24 to C47, C28 to C48, C52 to C49, C43 to C5, C54 to C50, C16 to C51, C18 to C52, C34 to C53, C36 to C54, C48 to C55, C12 to C56, C30 to C57, C38 to C58, C40 to C59, C49 to C6, C2 to C60, C4 to C61, C20 to C62, C22 to C63, C58 to C7, C61 to C8, C5 to C9, D3 to D2, D5 to D3, D7 to D4, D6 to D5, D2 to D6, D4 to D7, J3 to J2, J6 to J3, J8 to J4, J7 to J5, J2 to J6, J4 to J7, L3 to L2, L5 to L3, L7 to L4, L6 to L5, L2 to L6, L4 to L7, R9 to R10, R15 to R11, R20 to R12, R14 to R13, R2 to R14, R8 to R15, R18 to R16, R6 to R17, R12 to R18, R16 to R19, R7 to R2, R4 to R20, R10 to R21, R13 to R3, R19 to R4, R11 to R6, R17 to R7, R21 to R8, R3 to R9, U2 to U10, U7 to U11, U14 to U12, U4 to U13, U9 to U14, U6 to U2, U11 to U3, U16 to U4, U3 to U5, U8 to U6, U13 to U7, U17 to U8, U12 to U9, Y3 to Y2, Y5 to Y3, Y7 to Y4, Y6 to Y5, Y2 to Y6, Y4 to Y7
Connections:
- net GND: now also C64.2, C65.2, C66.2, J8.1 (Pin_1), R23.2, R24.2
- new net: U16.1 (OUT), U16.20 (OUT)
- new net: U16.10 (VSS), U16.11 (VSS), U16.21 (VSS)
- new net: U16.14 (VBAT), U16.15 (VBAT)
- new net: U16.18 (IN), U16.19 (IN)
- new net: J8.2 (Pin_2), Q1.2 (D)
- new net: C64.1, D8.1 (K), Q1.3 (S), U15.3 (VI)
- new net: C66.1, D9.2 (A), R22.2, R24.1, U15.1 (ADJ)
- new net: D8.2 (A), Q1.1 (G), R23.1
- new net DC: C65.1, D9.1 (K), R22.1, U15.2 (VO)
- no-connect marks 0 -> 1
Other:
- note added: "Power Supply"
- note removed: "To do:\n - Source the best capacitors/resistors for the RF section\n - Source the best voltage regulators & zenners for the RF section"

Commit message: Battery management for CVCO variant.
Parts:
- added BT1: 3.7V, Connector_Wire:SolderWirePad_1x02_P3.81mm_Drill1mm, symbol Device:Battery_Cell
- added C64: 10μF, Capacitor_SMD:C_0805_2012Metric_Pad1.15x1.40mm_HandSolder, symbol Device:C
- added C65, C66: 4.7μF, Capacitor_SMD:C_0805_2012Metric_Pad1.15x1.40mm_HandSolder, symbol Device:C
- added D10: Yellow, LED_THT:LED_D3.0mm_Horizontal_O1.27mm_Z2.0mm, symbol Device:LED
- added D8: Green, LED_THT:LED_D3.0mm_Horizontal_O1.27mm_Z2.0mm, symbol Device:LED
- added D9: Red, LED_THT:LED_D3.0mm_Horizontal_O1.27mm_Z2.0mm, symbol Device:LED
- added R22, R27, R29: 10k, Resistor_SMD:R_0805_2012Metric_Pad1.15x1.40mm_HandSolder, symbol Device:R
- added R23, R24, R25: 120, Resistor_SMD:R_0805_2012Metric_Pad1.15x1.40mm_HandSolder, symbol Device:R
- added R28: 1k, Resistor_SMD:R_0805_2012Metric_Pad1.15x1.40mm_HandSolder, symbol Device:R
- renumbered C64 to C67, C65 to C68, C66 to C69, D8 to D11, D9 to D12, R22 to R26, R23 to R30, R24 to R31
Connections:
- net DC: now also U16.18 (IN), U16.19 (IN), U16.2 (VPCC), C64.1, D10.2 (A), D8.2 (A), D9.2 (A), R22.1
- net GND: now also U16.10 (VSS), U16.11 (VSS), U16.21 (VSS), U16.9 (~TE), BT1.2 (-), C64.2, C65.2, C66.2, R27.2, R28.2, R29.2
- net BAT: now reaches U16.1 (OUT), U16.20 (OUT)
- net BAT: now also C66.1
- net at U16.12 (PROG3): now also R27.1
- net at U16.13 (PROG1): now also R28.1
- net at U16.14 (VBAT), U16.15 (VBAT): now also U16.16 (Vbat_SENSE), BT1.1 (+), C65.1
- net at U16.17 (CE): now also U16.3 (SEL), U16.4 (PROG2), R22.2
- net at U16.5 (THERM): now also R29.1
- net at U16.6 (~PG~): now also R23.2
- net at U16.7 (STAT2): now also R25.2
- net at U16.8 (STAT1/~LBO~): now also R24.2
- new net: D8.1 (K), R23.1
- new net: D9.1 (K), R24.1
- new net: D10.1 (K), R25.1
Other:
- note added: "Battery Management"
- moved on the sheet: C1, C10, C11, C12, C13, C14, C15, C16, C17, C18, C19, C2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

Commit message: 24V boost circuit added - CVCO.
Parts:
- added C72, C?: 4.7μF, Capacitor_SMD:C_0805_2012Metric_Pad1.15x1.40mm_HandSolder, symbol Device:C
- added L8: 10μH, Capacitor_SMD:C_0805_2012Metric_Pad1.15x1.40mm_HandSolder, symbol Device:L
- added R27: 3M, Resistor_SMD:R_0805_2012Metric_Pad1.15x1.40mm_HandSolder, symbol Device:R
- added R33: 100k, Resistor_SMD:R_0805_2012Metric_Pad1.15x1.40mm_HandSolder, symbol Device:R
- added U17: TPS61046, Package_TO_SOT_SMD:SOT-23-6_Handsoldering, symbol CVCO:TPS61040
- renumbered C67 to C68, C68 to C69, C69 to C71, D11 to D12, D12 to D13, R27 to R28, R28 to R29, R29 to R30, R30 to R31, R31 to R32
Connections:
- net BAT: now also C72.1, L8.2, U17.4 (EN), U17.5 (Vin)
- net GND: now also C72.2, C?.2, R33.2, U17.2 (GND)
- new net: R27.2, R33.1, U17.3 (FB)
- new net: L8.1, U17.1 (SW)
- new net VDD: C?.1, R27.1
- no-connect marks 1 -> 0
Other:
- note added: "24V Boost Circuit"
Changed lines of the file:
@@
 	1    0    0    -1
 $EndComp
-NoConn ~ 16050 13100
 Wire Wire Line
 	1400 13050 1400 13200
@@
 	4350 12600 4350 13050
 $Comp
-L Device:C C68
+L Device:C C69
 U 1 1 60DD8E2B
 P 4350 12450
-F 0 "C68" H 4465 12496 50  0000 L CNN
+F 0 "C69" H 4465 12496 50  0000 L CNN
 F 1 "1μF" H 4465 12405 50  0000 L CNN
 F 2 "Capacitor_SMD:C_0805_2012Metric_Pad1.15x1.40mm_HandSolder" H 4388 12300 50  0001 C CNN
@@
 	3900 12450 3900 12300
 $Comp
-L Device:D D12
+L Device:D D13
 U 1 1 60D0DB87
 P 3900 12150
-F 0 "D12" V 3854 12229 50  0000 L CNN
+F 0 "D13" V 3854 12229 50  0000 L CNN
 F 1 "1N4002" V 3945 12229 50  0000 L CNN
 F 2 "Diode_SMD:D_SMA_Handsoldering" H 3900 12150 50  0001 C CNN
@@
 	3000 12450 3000 12600
 $Comp
-L Device:R R31
+L Device:R R32
 U 1 1 608D6E34
 P 3000 12750
-F 0 "R31" H 3070 12796 50  0000 L CNN
+F 0 "R32" H 3070 12796 50  0000 L CNN
 F 1 "10k" H 3070 12705 50  0000 L CNN
 F 2 "Resistor_SMD:R_0805_2012Metric_Pad1.15x1.40mm_HandSolder" V 2930 12750 50  0001 C CNN
@@
 $EndComp
 $Comp
-L Device:C C69
+L Device:C C71
 U 1 1 606E00E9
 P 3450 12750
-F 0 "C69" H 3565 12796 50  0000 L CNN
+F 0 "C71" H 3565 12796 50  0000 L CNN
 F 1 "10μF" H 3565 12705 50  0000 L CNN
 F 2 "Capacitor_SMD:C_0805_2012Metric_Pad1.15x1.40mm_HandSolder" H 3488 12600 50  0001 C CNN
@@
 $EndComp
 $Comp
-L Device:C C67
+L Device:C C68
 U 1 1 606DFB5C
 P 2550 12450
-F 0 "C67" H 2665 12496 50  0000 L CNN
+F 0 "C68" H 2665 12496 50  0000 L CNN
 F 1 "0.1μF" H 2665 12405 50  0000 L CNN
 F 2 "Capacitor_SMD:C_0805_2012Metric_Pad1.15x1.40mm_HandSolder" H 2588 12300 50  0001 C CNN
@@
 	2100 11850 2100 12000
 $Comp
-L Device:D_Zener D11
+L Device:D_Zener D12
 U 1 1 615F9BF3
 P 2100 12150
-F 0 "D11" V 2054 12229 50  0000 L CNN
+F 0 "D12" V 2054 12229 50  0000 L CNN
 F 1 "3V" V 2145 12229 50  0000 L CNN
 F 2 "Package_TO_SOT_SMD:SOT-23" H 2100 12150 50  0001 C CNN
@@
 	1750 12900 1750 13050
 $Comp
-L Device:R R30
+L Device:R R31
 U 1 1 6107C237
 P 1750 12750
-F 0 "R30" H 1820 12796 50  0000 L CNN
+F 0 "R31" H 1820 12796 50  0000 L CNN
 F 1 "100k" H 1820 12705 50  0000 L CNN
 F 2 "Resistor_SMD:R_0805_2012Metric_Pad1.15x1.40mm_HandSolder" V 1680 12750 50  0001 C CNN
@@
 	5350 13050 5350 12600
 $Comp
-L Device:R R27
+L Device:R R28
 U 1 1 64CB99E6
 P 5350 12450
-F 0 "R27" H 5420 12496 50  0000 L CNN
+F 0 "R28" H 5420 12496 50  0000 L CNN
 F 1 "10k" H 5420 12405 50  0000 L CNN
 F 2 "Resistor_SMD:R_0805_2012Metric_Pad1.15x1.40mm_HandSolder" V 5280 12450 50  0001 C CNN
@@
 	7750 11900 7150 11900
 $Comp
-L Device:R R28
+L Device:R R29
 U 1 1 648B4D90
 P 5800 12450
-F 0 "R28" H 5870 12496 50  0000 L CNN
+F 0 "R29" H 5870 12496 50  0000 L CNN
 F 1 "1k" H 5870 12405 50  0000 L CNN
 F 2 "Resistor_SMD:R_0805_2012Metric_Pad1.15x1.40mm_HandSolder" V 5730 12450 50  0001 C CNN
@@
 	8450 12900 8450 13050
 $Comp
-L Device:R R29
+L Device:R R30
 U 1 1 61645D0E
 P 6250 12450
-F 0 "R29" H 6320 12496 50  0000 L CNN
+F 0 "R30" H 6320 12496 50  0000 L CNN
 F 1 "10k" H 6320 12405 50  0000 L CNN
 F 2 "Resistor_SMD:R_0805_2012Metric_Pad1.15x1.40mm_HandSolder" V 6180 12450 50  0001 C CNN
@@
 Text Notes 5150 10550 0    50   ~ 0
 Battery Management
+Text Notes 12650 11700 0    50   ~ 0
+24V Boost Circuit
+Wire Notes Line
+	15750 11750 12650 11750
+Text GLabel 15400 12050 2    50   Input ~ 0
+VDD
+Wire Wire Line
+	15300 12750 15300 13150
+Connection ~ 14850 13150
+Wire Wire Line
+	15300 12050 15300 12450
+Wire Wire Line
+	14850 12550 14850 12750
+$Comp
+L Device:R R27
+U 1 1 65E1B724
+P 14850 12400
+F 0 "R27" H 14920 12446 50  0000 L CNN
+F 1 "3M" H 14920 12355 50  0000 L CNN
+F 2 "Resistor_SMD:R_0805_2012Metric_Pad1.15x1.40mm_HandSolder" V 14780 12400 50  0001 C CNN
+F 3 "~" H 14850 12400 50  0001 C CNN
+F 4 "C17662" H 14850 12400 50  0001 C CNN "LCSC Part #"
+	1    14850 12400
+	1    0    0    -1
+$EndComp
+Wire Wire Line
+	14850 13100 14850 13150
+$Comp
+L Device:R R33
+U 1 1 65E1B72C
+P 14850 12950
+F 0 "R33" H 14920 12996 50  0000 L CNN
+F 1 "100k" H 14920 12905 50  0000 L CNN
+F 2 "Resistor_SMD:R_0805_2012Metric_Pad1.15x1.40mm_HandSolder" V 14780 12950 50  0001 C CNN
+F 3 "~" H 14850 12950 50  0001 C CNN
+F 4 "C149504" H 14850 12950 50  0001 C CNN "LCSC Part #"
+	1    14850 12950
+	1    0    0    -1
+$EndComp
+Connection ~ 14350 13150
+Connection ~ 14850 12750
+Wire Wire Line
+	14850 13150 14350 13150
+Wire Wire Line
+	14850 12750 14850 12800
+Wire Wire Line
+	14850 12750 14250 12750
+Wire Wire Line
+	14850 12050 14850 12250
+Wire Wire Line
+	13750 12050 13050 12050
+$Comp
+L Device:L L8
+U 1 1 65E1B744
+P 13900 12050
+F 0 "L8" V 13719 12050 50  0000 C CNN
+F 1 "10μH" V 13810 12050 50  0000 C CNN
+F 2 "Capacitor_SMD:C_0805_2012Metric_Pad1.15x1.40mm_HandSolder" H 13900 12050 50  0001 C CNN
+F 3 "~" H 13900 12050 50  0001 C CNN
+F 4 "C1046" V 13900 12050 50  0001 C CNN "LCSC Part #"
+	1    13900 12050
+	0    1    1    0
+$EndComp
+Connection ~ 13050 12550
+Wire Wire Line
+	13050 12050 13050 12550
+Wire Wire Line
+	14350 12050 14050 12050
+Wire Wire Line
+	14350 12550 14350 12050
+Wire Wire Line
+	14250 12550 14350 12550
+Wire Wire Line
+	13050 12700 13050 12550
+$Comp
+L Device:C C72
+U 1 1 65E1B751
+P 13050 12850
+F 0 "C72" H 13165 12896 50  0000 L CNN
+F 1 "4.7μF" H 13165 12805 50  0000 L CNN
+F 2 "Capacitor_SMD:C_0805_2012Metric_Pad1.15x1.40mm_HandSolder" H 13088 12700 50  0001 C CNN
+F 3 "~" H 13050 12850 50  0001 C CNN
+F 4 "C37818" H 13050 12850 50  0001 C CNN "LCSC Part #"
+	1    13050 12850
+	1    0    0    -1
+$EndComp
+Connection ~ 13450 12550
+Wire Wire Line
+	13050 12550 13450 12550
+Wire Wire Line
+	13050 13150 13050 13000
+Wire Wire Line
+	14350 13150 13050 13150
+Wire Wire Line
+	14350 12950 14350 13150
+Wire Wire Line
+	14250 12950 14350 12950
+Wire Wire Line
+	13450 12950 13550 12950
+Wire Wire Line
+	13450 12550 13450 12950
+Wire Wire Line
+	13550 12550 13450 12550
+Wire Wire Line
+	13050 12050 12950 12050
+Connection ~ 13050 12050
+Connection ~ 13050 13150
+Wire Wire Line
+	13050 13150 13050 13250
+$Comp
+L power:GND #PWR059
+U 1 1 65E1B76B
+P 13050 13250
+F 0 "#PWR059" H 13050 13000 50  0001 C CNN
+F 1 "GND" H 13055 13077 50  0000 C CNN
+F 2 "" H 13050 13250 50  0001 C CNN
+F 3 "" H 13050 13250 50  0001 C CNN
+	1    13050 13250
+	1    0    0    -1
+$EndComp
+Wire Notes Line
+	15750 11750 15750 13550
+Wire Notes Line
+	12650 11750 12650 13550
+Wire Notes Line
+	12650 13550 15750 13550
+Text GLabel 12950 12050 0    50   Input ~ 0
+BAT
+$Comp
+L CVCO:TPS61040 U17
+U 1 1 66093CD9
+P 13900 12750
+F 0 "U17" H 13900 13215 50  0000 C CNN
+F 1 "TPS61046" H 13900 13124 50  0000 C CNN
+F 2 "Package_TO_SOT_SMD:SOT-23-6_Handsoldering" H 13950 12300 50  0001 C CNN
+F 3 "https://datasheet.lcsc.com/szlcsc/2001152032_Texas-Instruments-TLV61046ADBVR_C464815.pdf" H 14050 12750 50  0001 C CNN
+F 4 "C464815" H 13900 12750 50  0001 C CNN "LCSC Part #"
+	1    13900 12750
+	1    0    0    -1
+$EndComp
+Wire Wire Line
+	14850 12050 15300 12050
+$Comp
+L Device:C C?
+U 1 1 6633DDEA
+P 15300 12600
+F 0 "C?" H 15415 12646 50  0000 L CNN
+F 1 "4.7μF" H 15415 12555 50  0000 L CNN
+F 2 "Capacitor_SMD:C_0805_2012Metric_Pad1.15x1.40mm_HandSolder" H 15338 12450 50  0001 C CNN
+F 3 "~" H 15300 12600 50  0001 C CNN
+F 4 "C37818" H 15300 12600 50  0001 C CNN "LCSC Part #"
+	1    15300 12600
+	1    0    0    -1
+$EndComp
+Wire Wire Line
+	15300 13150 14850 13150
+Wire Wire Line
+	15300 12050 15400 12050
+Connection ~ 15300 12050
 $EndSCHEMATC
