File: hardware-cvco/hardware.sch (KiCad schematic (older format))
At the start: 158 parts, among them J1 SMA, J2 SMA, J3 SMA, J4 SMA, J5 SMA, J6 SMA, J7 SMA, J8 DC, Q1 AOD403, U1 L78L05_SOT89, U10 L78L05_SOT89, U11 L78L08_SOT89, U12 NLB-310-T1, U13 NLB-310-T1, U14 NLB-310-T1, U15 LM317DCYR, U16 MCP73871-2AA, U17 TPS61046, U2 L78L12_SOT89, U3 L78L12_SOT89, U4 L78L10_SOT89, U5 NLB-310-T1, U6 NLB-310-T1, U7 NLB-310-T1, U8 NLB-310-T1, U9 L78L10_SOT89, Y1 CVCO55CW-0100-0200, Y2 CVCO55CW-0200-0500, Y3 CV55CW500-1000, Y4 CVCO55CW-1000-2000, Y5 CVCO55CW-3500-4500, Y6 CV55BE1600-3200, Y7 CVCO55CC-3180-3710

Commit message: VCO switcher.
Parts:
- added C43, C77: 1μF, Capacitor_SMD:C_0805_2012Metric_Pad1.15x1.40mm_HandSolder, symbol Device:C
- added C44, C78: 0.1μF, Capacitor_SMD:C_0805_2012Metric_Pad1.15x1.40mm_HandSolder, symbol Device:C
- added C67: 1nF, Capacitor_THT:C_Disc_D5.0mm_W2.5mm_P2.50mm, symbol Device:C
- added C68, C73: 220nF, Capacitor_THT:C_Disc_D9.0mm_W2.5mm_P5.00mm, symbol Device:C
- added C79, C80, C81: 0.1μF, Capacitor_THT:C_Disc_D5.0mm_W2.5mm_P2.50mm, symbol Device:C
- added C82: 1nF, Capacitor_THT:C_Disc_D5.0mm_W2.5mm_P5.00mm, symbol Device:C
- added C83, C84: 0.1uF, Capacitor_THT:C_Disc_D5.0mm_W2.5mm_P2.50mm, symbol Device:C
- added D13: 10V, Diode_THT:D_DO-35_SOD27_P7.62mm_Horizontal, symbol Device:D_Zener
- added J5: Pickit 2, symbol Connector_Generic:Conn_02x03_Counter_Clockwise
- added Q2: PN2222A, Package_TO_SOT_THT:TO-92_Inline, symbol Transistor_BJT:PN2222A
- added R23, R42: 4.7k, Resistor_THT:R_Axial_DIN0207_L6.3mm_D2.5mm_P7.62mm_Horizontal, symbol Device:R
- added R24, R35, R36: 10k, Resistor_THT:R_Axial_DIN0207_L6.3mm_D2.5mm_P7.62mm_Horizontal, symbol Device:R
- added R28, R40, R41: 15k, Resistor_THT:R_Axial_DIN0207_L6.3mm_D2.5mm_P7.62mm_Horizontal, symbol Device:R
- added R30: 100k, Resistor_THT:R_Axial_DIN0207_L6.3mm_D2.5mm_P7.62mm_Horizontal, symbol Device:R
- added R43, R49: 2k, Resistor_THT:R_Axial_DIN0207_L6.3mm_D2.5mm_P7.62mm_Horizontal, symbol Device:R
- added R44: 82k, Resistor_THT:R_Axial_DIN0207_L6.3mm_D2.5mm_P7.62mm_Horizontal, symbol Device:R
- added R45: 6.7k, Resistor_THT:R_Axial_DIN0207_L6.3mm_D2.5mm_P7.62mm_Horizontal, symbol Device:R
- added R46: 3.3k, Resistor_THT:R_Axial_DIN0207_L6.3mm_D2.5mm_P7.62mm_Horizontal, symbol Device:R
- added R47: 7.5, Resistor_THT:R_Axial_DIN0207_L6.3mm_D2.5mm_P7.62mm_Horizontal, symbol Device:R
- added R48: 100, Resistor_THT:R_Axial_DIN0207_L6.3mm_D2.5mm_P7.62mm_Horizontal, symbol Device:R
- added SW1: On/Off, Connector_Wire:SolderWirePad_1x02_P3.81mm_Drill1.2mm, symbol Switch:SW_SPST
- added U12: PIC12F675-ISN, Package_DIP:DIP-8_W7.62mm, symbol MCU_Microchip_PIC12:PIC12F675-ISN
- added U16: LM358, symbol Amplifier_Operational:LM358
- added U20: 74LS06, symbol 74xx:74LS06
- gave numbers to parts that had none: 1
- renumbered C43 to C45, C44 to C46, C45 to C47, C46 to C48, C47 to C49, C48 to C50, C49 to C51, C50 to C52, C51 to C53, C52 to C54, C53 to C55, C54 to C56, C55 to C57, C56 to C58, C57 to C59, C58 to C60, C59 to C61, C60 to C62, C61 to C63, C62 to C64, C63 to C65, C64 to C66, C65 to C69, C66 to C70, C68 to C71, C69 to C72, C71 to C75, C72 to C76, D12 to D11, D13 to D12, J5 to J6, J6 to J7, J7 to J8, J8 to J9, R23 to R25, R24 to R26, R25 to R27, R26 to R29, R27 to R31, R28 to R32, R29 to R33, R30 to R34, R31 to R37, R32 to R38, R33 to R39, U12 to U13, U13 to U14, U14 to U15, U15 to U17, U16 to U18, U17 to U19
Connections:
- net GND: now also C73.2, J5.3 (Pin_3), R30.1, R35.1, R41.1, SW1.1 (A), U12.8 (VSS), U16.4 (V-); no longer J9.1 (Pin_1)
- net Sweep: now also C67.1, C83.2, R30.2, R36.1, U16.7
- net VDD renamed P2_VDD
- net P2_VDD: now also C43.1, C44.1, C68.1, C77.1, C78.1, J5.2 (Pin_2), R24.2, R40.2, U16.8 (V+), U20.2
- new net: C77.2, C78.2, U20.14 (VCC)
- new net: J9.1 (Pin_1), SW1.2 (B)
- new net: C43.2, C44.2, U12.1 (VDD)
- new net: R48.1, R49.1
- new net: C83.1, R48.2
- new net: C84.1, R49.2
- new net: C67.2, R23.1, U16.5 (+)
- new net: R23.2, R28.1, U16.1
- new net: R28.2, R36.2, U16.3 (+)
- new net: C79.2, C82.2, R45.1
- new net: Q2.3 (C), R42.1, R45.2
- new net: Q2.1 (E), R47.2
- new net: C81.2, Q2.2 (B), R44.1, R46.2
- new net: C81.1, D13.1 (K), R43.1
- new net: C80.2, R42.2, R43.2, R44.2
- new net: R40.1, R41.2, U16.6 (-)
- new net GP0: J5.6 (Pin_6), U12.7 (GP0), U20.1
- new net GP1: J5.5 (Pin_5), U12.6 (GP1), U20.11, U20.13, U20.3, U20.5, U20.9
- new net GP2: U12.5 (GP2)
- new net GP3: J5.1 (Pin_1), U12.4 (GP3)
- new net GP4: U12.3 (GP4)
- new net GP5: U12.2 (GP5)
- new net Noise: C84.2
- new net VGND: C68.2, C73.1, R24.1, R35.2, U16.2 (-)
- new net Vss: C80.1, C82.1, D13.2 (A), R46.1, R47.1, U20.7 (GND)
- no-connect marks 0 -> 1
Other:
- note added: "Amplification - Stage I"
- note added: "Amplification - Stage II"
- note added: "Noise Source"
- note added: "Summer"
- note added: "Sweep Generator"
- note added: "VCO Switcher"

Commit message: IC buffer added.
Parts:
- removed C37, C39, C41, C5, C7: 1μ, Capacitor_SMD:C_0805_2012Metric_Pad1.15x1.40mm_HandSolder, symbol Device:C
- removed C38, C40, C42, C6, C8: 0.1u, Capacitor_SMD:C_0805_2012Metric_Pad1.15x1.40mm_HandSolder, symbol Device:C
- removed D3: 18V, Package_TO_SOT_SMD:SOT-23, symbol Device:D_Zener
- removed D4, D5, D6: 20V, Package_TO_SOT_SMD:SOT-23, symbol Device:D_Zener
- removed D7: 16V, Package_TO_SOT_SMD:SOT-23, symbol Device:D_Zener
- removed R13, R14, R15, R3, R4: 1k, Resistor_SMD:R_0805_2012Metric_Pad1.15x1.40mm_HandSolder, symbol Device:R
- added C? (x5): 0.1u, Capacitor_SMD:C_0805_2012Metric_Pad1.15x1.40mm_HandSolder, symbol Device:C
- added C? (x5): 1μ, Capacitor_SMD:C_0805_2012Metric_Pad1.15x1.40mm_HandSolder, symbol Device:C
- added D?: 18V, Package_TO_SOT_SMD:SOT-23, symbol Device:D_Zener
- added D? (x3): 20V, Package_TO_SOT_SMD:SOT-23, symbol Device:D_Zener
- added D?: 16V, Package_TO_SOT_SMD:SOT-23, symbol Device:D_Zener
- added R? (x5): 1k, Resistor_SMD:R_0805_2012Metric_Pad1.15x1.40mm_HandSolder, symbol Device:R
- U20: value 74LS06 -> 74LS07
Connections:
- net GND: now also C?.2, C?.2, C?.2, C?.2, C?.2, C?.2, C?.2, C?.2, C?.2, C?.2, D?.2 (A), D?.2 (A), D?.2 (A), D?.2 (A), D?.2 (A); no longer U4.2 (GND)
- net GP1: no longer U20.11, U20.13, U20.5, U20.9
- net GP2: now also U20.5
- net GP3: now also U20.9
- net GP4: now also U20.11
- net GP5: now also U20.13
- net P2_VDD: now also C3.1, U10.3 (IN), U11.3 (IN), U2.3 (IN), U20.10, U20.12, U20.4, U20.6, U20.8, U3.3 (IN), U9.3 (IN), C?.1, C?.1, C?.1, C?.1, C?.1
- net Sweep: now also R?.2, R?.2, R?.2, R?.2, R?.2
- net VCC: no longer C3.1, U10.3 (IN), U11.3 (IN), U2.3 (IN), U3.3 (IN), U4.3 (IN), U9.3 (IN)
- net VCC_3: now also C?.1
- net VCC_4: now also C?.1; no longer U11.1 (OUT), U9.1 (OUT)
- net VCC_5: now also C?.1
- net VCC_6: now also U11.1 (OUT), C?.1; no longer C45.1, C46.1, C51.1, C52.1, R16.1
- net VT_3: now also D?.1 (K), R?.1
- net VT_4: now also D?.1 (K), R?.1
- net VT_5: now also D?.1 (K), R?.1
- net VT_6: now also D?.1 (K), R?.1; no longer C60.1, C61.1, Y5.2 (VT)
- new net VCC_7: C45.1, C46.1, C51.1, C52.1, C?.1, R16.1, U9.1 (OUT)
- new net VT_7: C60.1, C61.1, D?.1 (K), R?.1, Y5.2 (VT)
Other:
- moved on the sheet: BT1, C1, C2, C3, C4, C43, C44, C45, C46, C47, C48, C49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

Commit message: Noise Source & Summer added.
Parts:
- removed C79, C80, C81: 0.1μF, Capacitor_THT:C_Disc_D5.0mm_W2.5mm_P2.50mm, symbol Device:C
- removed C82: 1nF, Capacitor_THT:C_Disc_D5.0mm_W2.5mm_P5.00mm, symbol Device:C
- removed R42: 4.7k, Resistor_THT:R_Axial_DIN0207_L6.3mm_D2.5mm_P7.62mm_Horizontal, symbol Device:R
- removed R43: 2k, Resistor_THT:R_Axial_DIN0207_L6.3mm_D2.5mm_P7.62mm_Horizontal, symbol Device:R
- removed R44: 82k, Resistor_THT:R_Axial_DIN0207_L6.3mm_D2.5mm_P7.62mm_Horizontal, symbol Device:R
- removed R45: 6.7k, Resistor_THT:R_Axial_DIN0207_L6.3mm_D2.5mm_P7.62mm_Horizontal, symbol Device:R
- removed R46: 3.3k, Resistor_THT:R_Axial_DIN0207_L6.3mm_D2.5mm_P7.62mm_Horizontal, symbol Device:R
- removed R47: 7.5, Resistor_THT:R_Axial_DIN0207_L6.3mm_D2.5mm_P7.62mm_Horizontal, symbol Device:R
- added C80, C81, C83: 0.1μF, symbol Device:C_Small
- added C84: 50pF, symbol Device:C_Small
- added C85, C87: 10μF, symbol Device:C_Small
- added C86: 1nF, symbol Device:C_Small
- added R42: 1k, symbol Device:R_Small
- added R44: 2k, symbol Device:R_Small
- added R45: 3.3k, symbol Device:R_Small
- added R47: 27k, symbol Device:R_Small
- added R48: 6.7k, symbol Device:R_Small
- added R49: 10, symbol Device:R_Small
- added U21: LM386, symbol Amplifier_Audio:LM386
- gave numbers to parts that had none: 20
- renumbered C77 to C43, C78 to C44, C43 to C45, C44 to C46, C45 to C51, C46 to C52, C51 to C57, C52 to C58, C58 to C59, C59 to C60, C57 to C61, C60 to C66, C61 to C67, C66 to C68, C67 to C69, C68 to C70, C69 to C71, C70 to C72, C71 to C73, C72 to C74, C73 to C75, C74 to C76, C75 to C77, C76 to C78, C83 to C79, C84 to C82, J7 to J5, J8 to J6, J6 to J7, J5 to J8, L6 to L5, L7 to L6, L5 to L7, R17 to R16, R18 to R17, R16 to R18, R20 to R19, R21 to R20, R19 to R21, R48 to R43, R49 to R46, U9 to U12, U12 to U13, U13 to U16, U16 to U17, U17 to U18, U18 to U19, U20 to U2, U19 to U20, U2 to U3, U3 to U4, U4 to U5, U5 to U6, U6 to U7, U7 to U8, U8 to U9, Y6 to Y5, Y7 to Y6, Y5 to Y7
Connections:
- net VCC is gone; now on net P2_VDD: C1.1, U1.3 (IN)
- net GND: now also Q2.1 (E), U2.7 (GND), U5.2 (GND), C85.1, C86.1, R45.2, R49.2, U21.2 (-), U21.4 (GND)
- net Noise: now also C84.1, U21.5
- net P2_VDD: now also U5.3 (IN), R42.2, R44.1
- net Sweep: no longer R1.2, R13.2, R14.2, R15.2, R2.2, R3.2, R4.2
- net Tuner: now reaches R43.1, R46.1
- net Tuner: now also R1.2, R13.2, R14.2, R15.2, R2.2, R3.2, R4.2
- net at Q2.3 (C): now also R44.2, R47.1, R48.2
- net at Q2.2 (B): now also D13.2 (A)
- net at D13.1 (K): now also C85.2, R47.2
- removed net Vss: D13.2 (A), U2.7 (GND)
- new net: C87.2, U21.1 (GAIN)
- new net: C83.1, U21.3 (+)
- new net: C80.1, C81.1, U21.6 (V+)
- new net: C87.1, U21.8 (GAIN)
- new net: C84.2, R49.1
- new net: C83.2, C86.2, R48.1
- new net: C80.2, C81.2, R42.1, R45.1
- no-connect marks 1 -> 2
Other:
- note removed: "Amplification - Stage I"
- note removed: "Amplification - Stage II"
- moved on the sheet: BT1, C1, C10, C11, C12, C13, C14, C15, C16, C17, C18, C19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

Commit message: Simplified CVCO design.
Parts:
- removed C1, C3, C37, C39, C41, C5, C7: 1μ, Capacitor_SMD:C_0805_2012Metric_Pad1.15x1.40mm_HandSolder, symbol Device:C
- removed C17, C19, C21, C23, C53, C55, C57: 0.1n, Capacitor_SMD:C_0805_2012Metric_Pad1.15x1.40mm_HandSolder, symbol Device:C
- removed C18, C20, C22, C24, C54, C56, C58: 1n, Capacitor_SMD:C_0805_2012Metric_Pad1.15x1.40mm_HandSolder, symbol Device:C
- removed C2, C38, C4, C40, C42, C6, C8: 0.1u, Capacitor_SMD:C_0805_2012Metric_Pad1.15x1.40mm_HandSolder, symbol Device:C
- removed L1, L2, L3, L4, L5, L6, L7: 470n, Inductor_SMD:L_0805_2012Metric_Pad1.15x1.40mm_HandSolder, symbol Device:L
- removed R10: 560, Resistor_SMD:R_0805_2012Metric_Pad1.15x1.40mm_HandSolder, symbol Device:R
- removed R11: 680, Resistor_SMD:R_0805_2012Metric_Pad1.15x1.40mm_HandSolder, symbol Device:R
- removed R12, R21: 470, Resistor_SMD:R_0805_2012Metric_Pad1.15x1.40mm_HandSolder, symbol Device:R
- removed R19, R9: 220, Resistor_SMD:R_0805_2012Metric_Pad1.15x1.40mm_HandSolder, symbol Device:R
- removed R20: 270, Resistor_SMD:R_0805_2012Metric_Pad1.15x1.40mm_HandSolder, symbol Device:R
- removed U1, U10: L78L05_SOT89, Package_TO_SOT_SMD:SOT-89-3, symbol Regulator_Linear:L78L05_SOT89
- removed U11: L78L08_SOT89, Package_TO_SOT_SMD:SOT-89-3, symbol Regulator_Linear:L78L08_SOT89
- removed U12, U5: L78L10_SOT89, Package_TO_SOT_SMD:SOT-89-3, symbol Regulator_Linear:L78L10_SOT89
- removed U3, U4: L78L12_SOT89, Package_TO_SOT_SMD:SOT-89-3, symbol Regulator_Linear:L78L12_SOT89
- added R? (x2): 3.8k, Resistor_SMD:R_0805_2012Metric_Pad1.15x1.40mm_HandSolder, symbol Device:R
- added R? (x9): 1k, Resistor_SMD:R_0805_2012Metric_Pad1.15x1.40mm_HandSolder, symbol Device:R
- added R? (x2): 1.4k, Resistor_SMD:R_0805_2012Metric_Pad1.15x1.40mm_HandSolder, symbol Device:R
- added R?: 2k, Resistor_SMD:R_0805_2012Metric_Pad1.15x1.40mm_HandSolder, symbol Device:R
- C69, C79, C82: footprint Capacitor_THT:C_Disc_D5.0mm_W2.5mm_P2.50mm -> Capacitor_SMD:C_0805_2012Metric_Pad1.15x1.40mm_HandSolder
- C70, C75: footprint Capacitor_THT:C_Disc_D9.0mm_W2.5mm_P5.00mm -> Capacitor_SMD:C_0805_2012Metric_Pad1.15x1.40mm_HandSolder
- C80, C81, C83, C84, C85, C86, C87: footprint (none) -> Capacitor_SMD:C_0805_2012Metric_Pad1.15x1.40mm_HandSolder
- D10, D8, D9: footprint LED_THT:LED_D3.0mm_Horizontal_O1.27mm_Z2.0mm -> Connector_Wire:SolderWirePad_1x02_P3.81mm_Drill1mm
- D13: footprint Diode_THT:D_DO-35_SOD27_P7.62mm_Horizontal -> Diode_SMD:D_SMA_Handsoldering
- J8: footprint (none) -> Connector_PinHeader_2.54mm:PinHeader_1x06_P2.54mm_Vertical
- R16, R5: value 82 -> 220; LCSC Part # C25329 -> (none)
- R17: value 120 -> 270; LCSC Part # C114244 -> (none)
- R18, R8: value 150 -> 470; LCSC Part # C25283 -> (none)
- R23, R24, R28, R30, R35, R36, R40, R41, R43, R46: footprint Resistor_THT:R_Axial_DIN0207_L6.3mm_D2.5mm_P7.62mm_Horizontal -> Resistor_SMD:R_0805_2012Metric_Pad1.15x1.40mm_HandSolder
- R42, R44, R45, R47, R48, R49: footprint (none) -> Resistor_SMD:R_0805_2012Metric_Pad1.15x1.40mm_HandSolder
- R6: value 180 -> 560; LCSC Part # C104048 -> (none)
- R7: value 180 -> 680; LCSC Part # C104048 -> (none)
- U17, U21: footprint (none) -> Package_SO:SO-8_5.3x6.2mm_P1.27mm
- U2: footprint (none) -> Package_SO:SOIC-14_3.9x8.7mm_P1.27mm
Connections:
- net GND: now also J1.1 (In), J2.1 (In), J3.1 (In), J4.1 (In), J5.1 (In), J6.1 (In), J7.1 (In), U14.3, U15.3, U16.3, U6.3, U7.3, U8.3, U9.3, Y1.14 (VCC), Y2.14 (VCC), Y3.14 (VCC), Y4.14 (VCC), Y5.14 (VCC), Y6.14 (VCC), Y7.14 (VCC), R?.2, R?.2, R?.2, R?.2, R?.2, R?.2, R?.2
- net P2_VDD: now also R?.2, R?.2, R?.2, R?.2, R?.2, R?.2, R?.2
- net VCC_1: now also R5.2, R?.1, R?.1; no longer C10.1, C9.1, R5.1
- net VCC_2: now also R6.2, R?.1, R?.1; no longer C11.1, C12.1, R6.1
- net VCC_3: now also R7.2, R?.1, R?.1; no longer C13.1, C14.1, R7.1
- net VCC_4: now also R8.2, R?.1, R?.1; no longer C15.1, C16.1, R8.1
- net VCC_5: now also R16.2, R?.1, R?.1; no longer C47.1, C48.1, R16.1
- net VCC_6: now also R17.2, R?.1, R?.1; no longer C49.1, C50.1, R17.1
- net VCC_7: now also R18.2, R?.1, R?.1; no longer C51.1, C52.1, R18.1
- new net: C10.1, C9.1, R5.1
- new net: C11.1, C12.1, R6.1
- new net: C13.1, C14.1, R7.1
- new net: C15.1, C16.1, R8.1
- new net: C47.1, C48.1, R16.1
- new net: C49.1, C50.1, R17.1
- new net: C51.1, C52.1, R18.1
Other:
- moved on the sheet: D1, R1

Commit message: LCSC part numbers assigned.
Parts:
- C10, C12, C14, C16, C30, C32, C34, C36, C48, C50, C52, C63, C65, C67: value 0.1n -> 0.1nF; LCSC Part # 0805 -> C159771
- C11, C13, C15, C29, C31, C33, C35, C47, C49, C51, C62, C64, C66, C9: value 1n -> 1nF; LCSC Part # 0805 -> C1791
- C43, C45: LCSC Part # 0805 -> C116352
- C44, C46: LCSC Part # 0805 -> C62912
- C70, C75: value 220nF -> 1μF; LCSC Part # (none) -> C116352
- C79, C82: LCSC Part # (none) -> C62912
- J8: footprint Connector_PinHeader_2.54mm:PinHeader_1x06_P2.54mm_Vertical -> Connector_PinSocket_2.54mm:PinSocket_1x06_P2.54mm_Vertical; LCSC Part # (none) -> C40877
- R12, R53: renamed from R?; LCSC Part # C17513 -> C17388
- R19, R20, R21, R50, R54, R55, R56: renamed from R?; LCSC Part # C25329 -> C17513
- R24, R35, R36: LCSC Part # (none) -> C55866
- R30: LCSC Part # (none) -> C149504
- R43: LCSC Part # (none) -> C17408
- R46: LCSC Part # (none) -> C17604
- R51, R9: renamed from R?; value 3.8k -> 3.9k; LCSC Part # C17513 -> C17614
- R52: renamed from R?; LCSC Part # C17513 -> C17604
- U13: LCSC Part # (none) -> C96100
- U17: LCSC Part # (none) -> C7950
- U2: LCSC Part # (none) -> C513513
- gave numbers to parts that had none: 2
Other:
- moved on the sheet: BT1, C10, C11, C12, C13, C14, C15, C16, C25, C26, C27, C28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

Commit message: RF section layout finished - CVCO.
Parts:
- BT1, D10, D8, D9: footprint Connector_Wire:SolderWirePad_1x02_P3.81mm_Drill1mm -> Connector_PinSocket_2.54mm:PinSocket_1x02_P2.54mm_Vertical
- D1, D2, D3, D4, D5, D6, D7: footprint Package_TO_SOT_SMD:SOT-23 -> Diode_SMD:D_MiniMELF
- J1, J2, J3, J4, J5, J6, J7: footprint Connector_Coaxial:SMA_Amphenol_132134_Vertical -> CVCO:SMA-Edge
- J9: footprint Connector_BarrelJack:BarrelJack_Wuerth_6941xx301002 -> Connector_Wire:SolderWirePad_1x02_P3.81mm_Drill1mm
- SW1: footprint Connector_Wire:SolderWirePad_1x02_P3.81mm_Drill1.2mm -> Connector_PinSocket_2.54mm:PinSocket_1x02_P2.54mm_Vertical
- renumbered C9 to C1, C26 to C10, C27 to C11, C28 to C12, C79 to C13, C29 to C14, C30 to C15, C31 to C16, C32 to C17, C33 to C18, C34 to C19, C10 to C2, C35 to C20, C36 to C21, C82 to C22, C43 to C23, C44 to C24, C45 to C25, C46 to C26, C47 to C27, C48 to C28, C49 to C29, C11 to C3, C50 to C30, C51 to C31, C52 to C32, C59 to C33, C60 to C34, C61 to C35, C76 to C36, C62 to C37, C63 to C38, C64 to C39, C12 to C4, C65 to C40, C66 to C41, C67 to C42, C78 to C43, C68 to C44, C69 to C45, C80 to C46, C81 to C47, C70 to C48, C71 to C49, C13 to C5, C72 to C50, C83 to C51, C73 to C52, C74 to C53, C75 to C54, C84 to C55, C85 to C56, C86 to C57, C77 to C58, C87 to C59, C14 to C6, C15 to C7, C16 to C8, C25 to C9, L8 to L1, R20 to R10, R21 to R11, R50 to R12, R5 to R13, R6 to R14, R7 to R15, R8 to R16, R43 to R17, R46 to R18, R13 to R19, R14 to R20, R15 to R21, R51 to R22, R52 to R23, R53 to R24, R54 to R25, R55 to R26, R56 to R27, R16 to R28, R17 to R29, R18 to R30, R39 to R32, R22 to R33, R42 to R34, R23 to R35, R24 to R36, R25 to R37, R26 to R38, R27 to R39, R44 to R40, R45 to R41, R28 to R42, R29 to R43, R30 to R44, R47 to R45, R48 to R46, R32 to R47, R33 to R48, R34 to R49, R9 to R5, R35 to R50, R36 to R51, R37 to R52, R38 to R53, R49 to R54, R40 to R55, R41 to R56, R10 to R6, R11 to R7, R12 to R8, R19 to R9, U2 to U1, U20 to U10, U17 to U11, U18 to U12, U19 to U13, U21 to U14, U6 to U2, U7 to U3, U8 to U4, U9 to U5, U13 to U6, U14 to U7, U15 to U8, U16 to U9
Connections:
- net GND: no longer J1.1 (In), J2.1 (In), J3.1 (In), J4.1 (In), J5.1 (In), J6.1 (In), J7.1 (In), U2.3, U3.3, U4.3, U5.3, U7.3, U8.3, U9.3, Y1.14 (VCC), Y2.14 (VCC), Y3.14 (VCC), Y4.14 (VCC), Y5.14 (VCC), Y6.14 (VCC), Y7.14 (VCC)
- net at C1.1, C2.1, R13.1: now also J1.1 (In), U2.3, Y1.14 (VCC)
- net at C3.1, C4.1, R14.1: now also J2.1 (In), U3.3, Y2.14 (VCC)
- net at C5.1, C6.1, R15.1: now also J3.1 (In), U4.3, Y3.14 (VCC)
- net at C7.1, C8.1, R16.1: now also J4.1 (In), U5.3, Y4.14 (VCC)
- net at C27.1, C28.1, R28.1: now also J5.1 (In), U7.3, Y5.14 (VCC)
- net at C29.1, C30.1, R29.1: now also J6.1 (In), U8.3, Y6.14 (VCC)
- net at C31.1, C32.1, R30.1: now also J7.1 (In), U9.3, Y7.14 (VCC)
Other:
- moved on the sheet: C1, C2, C27, C28, C29, C3, C30, C31, C32, C4, C5, C6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

Commit message: Added horizontal Molex footprint & 3D model.
Parts:
- BT1, D10, D8, D9, SW1: footprint Connector_PinSocket_2.54mm:PinSocket_1x02_P2.54mm_Vertical -> CVCO:2-2.54mm-Horizontal-Molex
- D1: value 5V -> 5.1V; LCSC Part # C455057 -> C305343
- D2, D3: LCSC Part # C85086 -> C268731
- D4, D5, D7: LCSC Part # C85086 -> C398899
- D6: LCSC Part # C85086 -> C313481
- Q2: value PN2222A -> MBT2222; footprint Package_TO_SOT_THT:TO-92_Inline -> Package_TO_SOT_SMD:SOT-23; LCSC Part # (none) -> C82460
Connections:
- net GND: now also SW1.2 (B); no longer SW1.1 (A)
- net at J9.1 (Pin_1): now also Q1.2 (D); no longer SW1.2 (B)
- net at J9.2 (Pin_2): now also SW1.1 (A); no longer Q1.2 (D)
Changed lines of the file:
@@
 encoding utf-8
 Sheet 1 1
-Title "Hide My Ass"
+Title "HideMyAss"
 Date "2020-08-24"
 Rev "1.0.0"
@@
 L Connector_Generic:Conn_01x02 J9
 U 1 1 6065063C
-P 1100 12200
-F 0 "J9" H 1018 11875 50  0000 C CNN
-F 1 "DC" H 1018 11966 50  0000 C CNN
-F 2 "Connector_Wire:SolderWirePad_1x02_P3.81mm_Drill1mm" H 1100 12200 50  0001 C CNN
-F 3 "~" H 1100 12200 50  0001 C CNN
-	1    1100 12200
-	-1   0    0    1
+P 1100 12100
+F 0 "J9" H 1018 11775 50  0000 C CNN
+F 1 "DC" H 1018 11866 50  0000 C CNN
+F 2 "Connector_Wire:SolderWirePad_1x02_P3.81mm_Drill1mm" H 1100 12100 50  0001 C CNN
+F 3 "~" H 1100 12100 50  0001 C CNN
+	1    1100 12100
+	-1   0    0    -1
 $EndComp
 $Comp
@@
 F 0 "D10" V 10489 11428 50  0000 L CNN
 F 1 "Yellow" V 10398 11428 50  0000 L CNN
-F 2 "Connector_PinSocket_2.54mm:PinSocket_1x02_P2.54mm_Vertical" H 10450 11350 50  0001 C CNN
+F 2 "CVCO:2-2.54mm-Horizontal-Molex" H 10450 11350 50  0001 C CNN
 F 3 "~" H 10450 11350 50  0001 C CNN
 	1    10450 11350
@@
 F 0 "D9" V 10039 11428 50  0000 L CNN
 F 1 "Red" V 9948 11428 50  0000 L CNN
-F 2 "Connector_PinSocket_2.54mm:PinSocket_1x02_P2.54mm_Vertical" H 10000 11350 50  0001 C CNN
+F 2 "CVCO:2-2.54mm-Horizontal-Molex" H 10000 11350 50  0001 C CNN
 F 3 "~" H 10000 11350 50  0001 C CNN
 	1    10000 11350
 	0    1    -1   0
 $EndComp
-$Comp
-L Device:LED D8
-U 1 1 629E6AE0
-P 9550 11350
-F 0 "D8" V 9589 11428 50  0000 L CNN
-F 1 "Green" V 9498 11428 50  0000 L CNN
-F 2 "Connector_PinSocket_2.54mm:PinSocket_1x02_P2.54mm_Vertical" H 9550 11350 50  0001 C CNN
-F 3 "~" H 9550 11350 50  0001 C CNN
-	1    9550 11350
-	0    1    -1   0
-$EndComp
 Connection ~ 10000 11050
 Wire Wire Line
@@
 F 0 "BT1" H 11518 12396 50  0000 L CNN
 F 1 "3.7V" H 11518 12305 50  0000 L CNN
-F 2 "Connector_PinSocket_2.54mm:PinSocket_1x02_P2.54mm_Vertical" V 11400 12360 50  0001 C CNN
+F 2 "CVCO:2-2.54mm-Horizontal-Molex" V 11400 12360 50  0001 C CNN
 F 3 "~" V 11400 12360 50  0001 C CNN
 	1    11400 12300
@@
 Wire Wire Line
 	1450 12950 1450 13300
-$Comp
-L Switch:SW_SPST SW1
-U 1 1 60C7FD23
-P 1450 12750
-F 0 "SW1" V 1496 12662 50  0000 R CNN
-F 1 "On/Off" V 1405 12662 50  0000 R CNN
-F 2 "Connector_PinSocket_2.54mm:PinSocket_1x02_P2.54mm_Vertical" H 1450 12750 50  0001 C CNN
-F 3 "" H 1450 12750 50  0001 C CNN
-	1    1450 12750
-	0    1    -1   0
-$EndComp
 Wire Wire Line
 	15600 9250 15450 9250
@@
 	1    0    0    -1
 $EndComp
-Text GLabel 17250 10150 0    50   Input ~ 0
-P2_VPP
 Wire Wire Line
 	17400 10150 17250 10150
@@
 P 19650 13050
 F 0 "Q2" H 19840 13096 50  0000 L CNN
-F 1 "PN2222A" H 19840 13005 50  0000 L CNN
-F 2 "Package_TO_SOT_THT:TO-92_Inline" H 19850 12975 50  0001 L CIN
-F 3 "http://www.fairchildsemi.com/ds/PN/PN2222A.pdf" H 19650 13050 50  0001 L CNN
+F 1 "MBT2222" H 19840 13005 50  0000 L CNN
+F 2 "Package_TO_SOT_SMD:SOT-23" H 19850 12975 50  0001 L CIN
+F 3 "https://datasheet.lcsc.com/szlcsc/1809272022_ON-Semiconductor-MMBT2222ALT1G_C82460.pdf" H 19650 13050 50  0001 L CNN
+F 4 "C82460" H 19650 13050 50  0001 C CNN "LCSC Part #"
 	1    19650 13050
 	1    0    0    -1
@@
 P 1900 1950
 F 0 "D1" V 1854 2029 50  0000 L CNN
-F 1 "5V" V 1945 2029 50  0000 L CNN
+F 1 "5.1V" V 1945 2029 50  0000 L CNN
 F 2 "Diode_SMD:D_MiniMELF" H 1900 1950 50  0001 C CNN
 F 3 "~" H 1900 1950 50  0001 C CNN
-F 4 "C455057" V 1900 1950 50  0001 C CNN "LCSC Part #"
+F 4 "C305343" V 1900 1950 50  0001 C CNN "LCSC Part #"
 	1    1900 1950
 	0    1    1    0
@@
 F 2 "Diode_SMD:D_MiniMELF" H 11300 6750 50  0001 C CNN
 F 3 "~" H 11300 6750 50  0001 C CNN
-F 4 "C85086" V 11300 6750 50  0001 C CNN "LCSC Part #"
+F 4 "C398899" V 11300 6750 50  0001 C CNN "LCSC Part #"
 	1    11300 6750
 	0    1    1    0
@@
 F 2 "Diode_SMD:D_MiniMELF" H 6600 6750 50  0001 C CNN
 F 3 "~" H 6600 6750 50  0001 C CNN
-F 4 "C85086" V 6600 6750 50  0001 C CNN "LCSC Part #"
+F 4 "C313481" V 6600 6750 50  0001 C CNN "LCSC Part #"
 	1    6600 6750
 	0    1    1    0
@@
 F 2 "Diode_SMD:D_MiniMELF" H 1900 6750 50  0001 C CNN
 F 3 "~" H 1900 6750 50  0001 C CNN
-F 4 "C85086" V 1900 6750 50  0001 C CNN "LCSC Part #"
+F 4 "C398899" V 1900 6750 50  0001 C CNN "LCSC Part #"
 	1    1900 6750
 	0    1    1    0
@@
 F 2 "Diode_SMD:D_MiniMELF" H 16000 2000 50  0001 C CNN
 F 3 "~" H 16000 2000 50  0001 C CNN
-F 4 "C85086" V 16000 2000 50  0001 C CNN "LCSC Part #"
+F 4 "C398899" V 16000 2000 50  0001 C CNN "LCSC Part #"
 	1    16000 2000
 	0    1    1    0
@@
 F 2 "Diode_SMD:D_MiniMELF" H 11300 2000 50  0001 C CNN
 F 3 "~" H 11300 2000 50  0001 C CNN
-F 4 "C85086" V 11300 2000 50  0001 C CNN "LCSC Part #"
+F 4 "C268731" V 11300 2000 50  0001 C CNN "LCSC Part #"
 	1    11300 2000
 	0    1    1    0
@@
 F 2 "Diode_SMD:D_MiniMELF" H 6600 1950 50  0001 C CNN
 F 3 "~" H 6600 1950 50  0001 C CNN
-F 4 "C85086" V 6600 1950 50  0001 C CNN "LCSC Part #"
+F 4 "C268731" V 6600 1950 50  0001 C CNN "LCSC Part #"
 	1    6600 1950
 	0    1    1    0
@@
 	6450 1650 6600 1650
 Connection ~ 6600 1650
+$Comp
+L Switch:SW_SPST SW1
+U 1 1 60C7FD23
+P 1450 12750
+F 0 "SW1" V 1496 12662 50  0000 R CNN
+F 1 "On/Off" V 1405 12662 50  0000 R CNN
+F 2 "CVCO:2-2.54mm-Horizontal-Molex" H 1450 12750 50  0001 C CNN
+F 3 "" H 1450 12750 50  0001 C CNN
+	1    1450 12750
+	0    1    1    0
+$EndComp
+$Comp
+L Device:LED D8
+U 1 1 629E6AE0
+P 9550 11350
+F 0 "D8" V 9589 11428 50  0000 L CNN
+F 1 "Green" V 9498 11428 50  0000 L CNN
+F 2 "CVCO:2-2.54mm-Horizontal-Molex" H 9550 11350 50  0001 C CNN
+F 3 "~" H 9550 11350 50  0001 C CNN
+	1    9550 11350
+	0    1    -1   0
+$EndComp
+Text GLabel 17250 10150 0    50   Input ~ 0
+P2_VPP
 $EndSCHEMATC

Commit message: Rough layout of the non-RF section.
Parts:
- added F1: 3A Fast, Fuse:Fuse_1206_3216Metric_Pad1.42x1.75mm_HandSolder, symbol Device:Fuse
- D11: value 3V -> 10V; footprint Package_TO_SOT_SMD:SOT-23 -> Diode_SMD:D_MiniMELF; LCSC Part # C118562 -> C398894
- D13: footprint Diode_SMD:D_SMA_Handsoldering -> Diode_SMD:D_MiniMELF; LCSC Part # (none) -> C398894
- U6: footprint Package_DIP:DIP-8_W7.62mm -> Package_SO:SOIC-8_3.9x4.9mm_P1.27mm
Connections:
- net at J9.1 (Pin_1): now also F1.1; no longer Q1.2 (D)
- new net: F1.2, Q1.2 (D)
Other:
- moved on the sheet: BT1, C1, C10, C11, C12, C13, C14, C15, C16, C17, C18, C19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
