File: hardware-cvco/hardware.kicad_pcb (KiCad board)
At the start: 4 copper layers, 99 x 80 mm, 170 parts, among them J1 SMA, J2 SMA, J3 SMA, J4 SMA, J5 SMA, J6 SMA, J7 SMA, J8 Pickit 2, J9 DC, Q1 AOD403, Q2 MBT2222, SW1 On/Off, U1 74LS07, U10 TPS61046, U11 BQ21040, U12 LM324, U13 LM317DCYR, U14 LM386, U2 NLB-310-T1, U3 NLB-310-T1, U4 NLB-310-T1, U5 NLB-310-T1, U6 PIC12F675-ISN, U7 NLB-310-T1, U8 NLB-310-T1, U9 NLB-310-T1, Y1 CVCO55CW-0100-0200, Y2 CVCO55CW-0200-0500, Y3 CV55CW500-1000, Y4 CVCO55CW-1000-2000, Y5 CV55BE1600-3200, Y6 CVCO55CC-3180-3710, Y7 CVCO55CW-3500-4500

Commit message: Boost circuit update.
Parts:
- removed G*** (x2): Lightbulb, Icons:Lightbulb
- removed G***: Thermometer, Icons:Thermometer
- removed G***: Battery, Icons:Battery
- removed G***: Switch, Icons:Switch
- removed G***: Lightning, Icons:Lightning
- removed R13, R28: 220, Resistor_SMD:R_0805_2012Metric_Pad1.15x1.40mm_HandSolder
- removed R14: 560, Resistor_SMD:R_0805_2012Metric_Pad1.15x1.40mm_HandSolder
- removed R15: 680, Resistor_SMD:R_0805_2012Metric_Pad1.15x1.40mm_HandSolder
- removed R16, R30: 470, Resistor_SMD:R_0805_2012Metric_Pad1.15x1.40mm_HandSolder
- removed R29: 270, Resistor_SMD:R_0805_2012Metric_Pad1.15x1.40mm_HandSolder
- C54: value 50pF -> 47pF
- D11: footprint Diode_SMD:D_SMA_Handsoldering -> Diode_SMD:D_SMA
- R45: value 6.7k -> 6.8k
Connections:
- C1 pad 1: Net-(C1-Pad1) -> VCC_1
- C2 pad 1: Net-(C1-Pad1) -> VCC_1
- C27 pad 1: Net-(C27-Pad1) -> VCC_5
- C28 pad 1: Net-(C27-Pad1) -> VCC_5
- C29 pad 1: Net-(C29-Pad1) -> VCC_6
- C3 pad 1: Net-(C3-Pad1) -> VCC_2
- C30 pad 1: Net-(C29-Pad1) -> VCC_6
- C31 pad 1: Net-(C31-Pad1) -> VCC_7
- C32 pad 1: Net-(C31-Pad1) -> VCC_7
- C4 pad 1: Net-(C3-Pad1) -> VCC_2
- C5 pad 1: Net-(C5-Pad1) -> VCC_3
- C52 pad 1: DC -> VDD
- C6 pad 1: Net-(C5-Pad1) -> VCC_3
- C7 pad 1: Net-(C7-Pad1) -> VCC_4
- C8 pad 1: Net-(C7-Pad1) -> VCC_4
- D11 pad 1: DC -> VDD
- J1 pad 1: Net-(C1-Pad1) -> VCC_1
- J2 pad 1: Net-(C3-Pad1) -> VCC_2
- J3 pad 1: Net-(C5-Pad1) -> VCC_3
- J4 pad 1: Net-(C7-Pad1) -> VCC_4
- J5 pad 1: Net-(C27-Pad1) -> VCC_5
- J6 pad 1: Net-(C29-Pad1) -> VCC_6
- J7 pad 1: Net-(C31-Pad1) -> VCC_7
- R42 pad 1: DC -> VDD
- U10 pad 5: BAT -> Boost
- U10 pad 6: (no net) -> BAT
- U13 pad 2: DC -> VDD
- U2 pad 3: Net-(C1-Pad1) -> VCC_1
- U3 pad 3: Net-(C3-Pad1) -> VCC_2
- U4 pad 3: Net-(C5-Pad1) -> VCC_3
- U5 pad 3: Net-(C7-Pad1) -> VCC_4
- U7 pad 3: Net-(C27-Pad1) -> VCC_5
- U8 pad 3: Net-(C29-Pad1) -> VCC_6
- U9 pad 3: Net-(C31-Pad1) -> VCC_7
- Y1 pad 14: Net-(C1-Pad1) -> VCC_1
- Y2 pad 14: Net-(C3-Pad1) -> VCC_2
- Y3 pad 14: Net-(C5-Pad1) -> VCC_3
- Y4 pad 14: Net-(C7-Pad1) -> VCC_4
- Y5 pad 14: Net-(C27-Pad1) -> VCC_5
- Y6 pad 14: Net-(C29-Pad1) -> VCC_6
- Y7 pad 14: Net-(C31-Pad1) -> VCC_7
Routing:
- net VDD: track 91.8 -> 139.5 mm
- net VCC_7: track 6.09 -> 50.2 mm
- net VCC_6: track 6.09 -> 50.1 mm
- net VCC_5: track 6.09 -> 50.1 mm
- net VCC_1: track 6.10 -> 48.4 mm
- net VCC_2: track 6.08 -> 48.4 mm
- net VCC_4: track 6.08 -> 48.3 mm
- net VCC_3: track 6.08 -> 48.3 mm
- net Net-(C31-Pad1): track 42.0 -> 0.00 mm
- net Net-(C29-Pad1): track 42.0 -> 0.00 mm
- net Net-(C27-Pad1): track 42.0 -> 0.00 mm
- net Net-(C1-Pad1): track 40.3 -> 0.00 mm
- net Net-(C3-Pad1): track 40.2 -> 0.00 mm
- net Net-(C7-Pad1): track 40.2 -> 0.00 mm
- net Net-(C5-Pad1): track 40.2 -> 0.00 mm
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Other:
- board text added: "Rev 1.0.1"
- board text removed: "Rev 1.0.0"
