File: hardware-discrete/hardware-discrete.sch (KiCad schematic (older format))
At the start: 65 parts, among them J1 5V, J2 Pickit 2, Q1 FQP13N06L, Q2 BD137, Q3 BD137, Q4 BD137, SW1 On/Off, U1 LM317, U2 NE555, U3 TL064, U4 L7805, U5 PIC12F675-IP

Commit message: Power Supply & Battery Management update.
Parts:
- removed U3: TL064, Package_DIP:DIP-14_W7.62mm_Socket, symbol Amplifier_Operational:TL064
- added C20: 1μF, symbol Device:CP
- added C21: 0.1μF, symbol Device:CP
- added C22: 25pF, symbol Device:C
- added C23: 10nF, Capacitor_THT:C_Disc_D5.0mm_W2.5mm_P2.50mm, symbol Device:C
- added D10, D11, D8, D9: 1N4007, Diode_THT:D_DO-41_SOD81_P7.62mm_Horizontal, symbol Device:D
- added F1: 1.5A Fast, symbol Device:Fuse
- added JP1: Safety Net, Connector_PinHeader_2.54mm:PinHeader_1x02_P2.54mm_Vertical, symbol Device:Jumper_NC_Small
- added M1: Fan, symbol Motor:Fan
- added R26: 60, Resistor_THT:R_Axial_DIN0617_L17.0mm_D6.0mm_P5.08mm_Vertical, symbol Device:R
- added R27: 33, symbol Device:R
- added SW2: F/S Mode, symbol Switch:SW_SPDT
- added TH1: 10k, symbol Device:Thermistor_NTC
- added U3: LM7824_TO220, Package_TO_SOT_THT:TO-220-3_Vertical, symbol Regulator_Linear:LM7824_TO220
- added U6: LM358, symbol Amplifier_Operational:LM358
- C14, C15, C17, C18, C19: footprint (none) -> Capacitor_THT:CP_Radial_D5.0mm_P2.00mm
- C16: value 10nF -> 1nF
- D1, D3, D4: value 1N4001 -> 1N4007; footprint (none) -> Diode_THT:D_DO-41_SOD81_P7.62mm_Horizontal
- D2: footprint (none) -> Diode_THT:D_DO-41_SOD81_P7.62mm_Horizontal
- D5, D6: footprint (none) -> Connector_PinHeader_2.54mm:PinHeader_1x02_P2.54mm_Vertical
- D7: value GREEN -> BLUE; footprint (none) -> Connector_PinHeader_2.54mm:PinHeader_1x02_P2.54mm_Vertical
- J1: value 5V -> 24V
- J2: footprint (none) -> Connector_PinHeader_2.54mm:PinHeader_1x03_P2.54mm_Vertical
- R10: value 820 -> 680; footprint (none) -> Resistor_THT:R_Axial_DIN0207_L6.3mm_D2.5mm_P7.62mm_Horizontal
- R11, R18, R20, R21: footprint (none) -> Resistor_THT:R_Axial_DIN0207_L6.3mm_D2.5mm_P7.62mm_Horizontal
- R13, R16, R22, R9: footprint (none) -> Resistor_THT:R_Axial_DIN0516_L15.5mm_D5.0mm_P5.08mm_Vertical
- R19: value 10 -> 18; footprint (none) -> Resistor_THT:R_Axial_DIN0516_L15.5mm_D5.0mm_P5.08mm_Vertical
- R2: value 1k -> 1.2k
- R23: value 18 -> 33; footprint (none) -> Resistor_THT:R_Axial_DIN0516_L15.5mm_D5.0mm_P5.08mm_Vertical
- R5: value 560 -> 470
- R8: footprint (none) -> Resistor_THT:R_Axial_DIN0617_L17.0mm_D6.0mm_P5.08mm_Vertical
- U4: footprint (none) -> Package_TO_SOT_THT:TO-220-3_Vertical
- gave numbers to parts that had none: 4
Connections:
- net labels added: BREF
- wire segments 234 -> 271
Other:
- note added: "12V Regulator"
- note added: "24V Boost Circuit"
- note added: "Temperature Control"
- note removed: "30V Boost Circuit"
- note removed: "5V Regulator"
- note removed: "Unused Op-Amp"
- moved on the sheet: BT1, C1, C10, C11, C12, C13, C16, C17, C18, C19, C2, C3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

Commit message: Temperature control.
Parts:
- removed D11, D9: 1N4007, Diode_THT:D_DO-41_SOD81_P7.62mm_Horizontal, symbol Device:D
- removed Q3: BD137, Package_TO_SOT_THT:TO-126-3_Vertical, symbol Transistor_BJT:BD137
- added D?: 5.2V, symbol Device:D_Zener
- added Q?: BD137, Package_TO_SOT_THT:TO-126-3_Vertical, symbol Transistor_BJT:BD137
- added Q?: 2N3904, Package_TO_SOT_THT:TO-92_Inline, symbol Transistor_BJT:2N3904
- added R?: 1k, Resistor_THT:R_Axial_DIN0516_L15.5mm_D5.0mm_P5.08mm_Vertical, symbol Device:R
- added R? (x5): 10k, symbol Device:R
- added R?: 20k, symbol Device:R
- added R?: 8k, symbol Device:R
- added U? (x3): LM393, symbol Comparator:LM393
- J1: value 24V -> 12V
- R10: value 680 -> 820
- R11: value 1.2k -> 10k
- R2: value 1.2k -> 240
- R23, R27, R9: value 33 -> 56
- R26, R8: value 60 -> 56
- R5: value 470 -> 390
- R6: value 10k -> 1.7k
Connections:
- net BAT: now also Q?.3 (C)
- net DC: now also TH1.1, R?.1, R?.1, R?.1, U?.8 (V+)
- net GND: now also M1.2 (-), Q?.1 (E), R?.1, R?.2, R?.2, R?.2, U?.4 (V-); no longer C17.2, C18.2, U4.2 (GND)
- net at M1.1 (+): now also R?.1, R?.1, R?.2, R?.2, U?.1, U?.7
- net at TH1.2: now also R?.2, U?.3 (+), U?.6 (_)
- net at D1.1 (K), D3.1 (K), U1.3 (VI): now also C10.1
- net at R16.2: now also Q?.1 (E)
- net at R11.1: now also Q?.2 (B)
- net at C17.1, SW1.2 (B), U4.1 (IN): now also R?.2
- net CHG: no longer names the net of D10.2 (A), R19.1, R23.2
- new net: C17.2, C18.2, Q?.2 (C), U4.2 (GND)
- new net: D?.2 (A), Q?.3 (B)
- new net: D?.1 (K), R?.1
- new net: R?.1, R?.2, U?.2 (-), U?.5 (+)
Other:
- note added: "10V Regulator"
- note added: "High Speed"
- note added: "Low Speed"
- note removed: "12V Regulator"
- moved on the sheet: BT1, C16, C17, C18, C19, C23, D10, D7, JP1, M1, Q4, R12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

Commit message: Battery management update.
Parts:
- removed J2: Pickit 2, Connector_PinHeader_2.54mm:PinHeader_1x03_P2.54mm_Vertical, symbol Connector_Generic:Conn_01x03
- removed Q?: 2N3904, Package_TO_SOT_THT:TO-92_Inline, symbol Transistor_BJT:2N3904
- added C24, C26: 1μF, symbol Device:CP
- added C25, C27: 0.1μF, symbol Device:CP
- added J2: Conn_01x05, symbol Connector_Generic:Conn_01x05
- added JP? (x2): MCU Isolation, Connector_PinHeader_2.54mm:PinHeader_1x02_P2.54mm_Vertical, symbol Device:Jumper_NC_Small
- added Q?: BD137, Package_TO_SOT_THT:TO-126-3_Vertical, symbol Transistor_BJT:BD137
- added R36: 470, Resistor_THT:R_Axial_DIN0516_L15.5mm_D5.0mm_P5.08mm_Vertical, symbol Device:R
- added R?: 2.2, Resistor_THT:R_Axial_DIN0516_L15.5mm_D5.0mm_P5.08mm_Vertical, symbol Device:R
- D4: renamed from D2; value 1N4001 -> 1N4007
- D7: renamed from D?; value 5.2V -> 2.6V
- M1: value Fan -> 5V
- R10: renamed from R27; value 56 -> 62
- R11: renamed from R9; value 56 -> 62
- R2: value 240 -> 100
- R24: renamed from R19; value 18 -> 10
- R26: renamed from R23; value 56 -> 120
- R8: value 56 -> 62
- R9: renamed from R26; value 56 -> 62
- gave numbers to parts that had none: 10
- renumbered C8 to C10, C9 to C11, C10 to C12, C22 to C13, C11 to C14, C12 to C15, C13 to C16, C16 to C17, C14 to C18, C15 to C19, C23 to C20, C17 to C21, C18 to C22, C19 to C23, C20 to C8, C21 to C9, D7 to D10, D8 to D2, D4 to D5, D5 to D6, D6 to D8, D10 to D9, Q2 to Q3, Q4 to Q5, R11 to R12, R10 to R13, R12 to R14, R16 to R15, R13 to R16, R15 to R18, R14 to R19, R17 to R20, R18 to R21, R24 to R22, R25 to R23, R21 to R25, R22 to R27, R20 to R28, SW2 to SW1, SW1 to SW2, U3 to U2, U2 to U3, U6 to U4, U4 to U6
Connections:
- net Boost is gone; now on net BOOST: C9.1, U2.3 (VO)
- net BREF: now also J2.4 (Pin_4), JP?.1; no longer R10.2, R9.1
- net DC: now also R36.2; no longer U7.8 (V+)
- net GND: now also C24.2, C25.2, C26.2, C27.2, J2.5 (Pin_5); no longer BT1.2 (-), C23.2, Q4.1 (E), R28.1
- net PWM: now also U3.3 (Q)
- net PWR: no longer U3.3 (Q)
- net S1: now also J2.3 (Pin_3)
- net S3: now also J2.1 (Pin_1)
- net at M1.1 (+), R30.2, R32.1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: now also C26.1, C27.1
- net at BT1.1 (+), C23.1, JP1.2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: now also R9.2
- net at R15.2: now also Q?.1 (E)
- net at R12.1: now also Q?.3 (B)
- net at C18.1, C19.1, R11.2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: now also JP?.2; no longer U5.1 (VDD)
- removed net BAT: D9.1 (K), JP1.1, Q3.2 (C), Q5.2 (C), R9.2
- net Sweep renamed SWEEP
- new net: JP?.2, R10.2, R9.1
- new net: Q4.1 (E), R?.2
- new net: C24.1, C25.1, R36.1, U7.8 (V+)
- new net BGND: BT1.2 (-), C23.2, Q3.2 (C), Q5.2 (C), Q?.2 (C), R28.1, R?.1
- new net CHG: D9.1 (K), JP1.1
- new net VDD: J2.2 (Pin_2), JP?.1, U5.1 (VDD)
Other:
- note added: "9V Regulator"
- note added: "Note: Arrangement will be altered to match the Pickit one."
- note added: "Pickit: 1-2-5-4-3"
- note removed: "10V Regulator"
- note removed: "VPP-DAT-CLK"
- moved on the sheet: BT1, C21, C22, C23, D10, D7, JP1, M1, Q4, R10, R17, R28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

Commit message: Charging switch.
Parts:
- removed C12: 0.1μF, symbol Device:CP
- removed C13: 25pF, symbol Device:C
- removed C14: 1μF, symbol Device:CP
- removed D1, D5: 1N4007, Diode_THT:D_DO-41_SOD81_P7.62mm_Horizontal, symbol Device:D
- removed R2: 100, symbol Device:R
- removed R6: 1.7k, symbol Device:R
- removed U1: LM317, symbol Regulator_Linear:LM317_3PinPackage
- added C?: 1μF, symbol Device:CP
- added C?: 0.1μF, symbol Device:CP
- added Q?: BD136, Package_TO_SOT_THT:TO-126-3_Vertical, symbol Transistor_BJT:BD136
- added Q?: 2N3904, Package_TO_SOT_THT:TO-92_Inline, symbol Transistor_BJT:2N3904
- added R?: 670, Resistor_THT:R_Axial_DIN0207_L6.3mm_D2.5mm_P7.62mm_Horizontal, symbol Device:R
- added R?: 1000, Resistor_THT:R_Axial_DIN0516_L15.5mm_D5.0mm_P5.08mm_Vertical, symbol Device:R
- added U?: L7809, symbol Regulator_Linear:L7809
- R10: value 62 -> 180
- R26: value 120 -> 62
Connections:
- net BGND: now also R10.1
- net CHG: now also Q?.2 (C); no longer D9.1 (K)
- net DC: now also C?.1, U?.3 (OUT)
- net GND: now also C?.2, C?.2, Q?.1 (E), U?.2 (GND); no longer R10.1
- net S1: now also R13.1; no longer R13.2
- net at Q?.3 (B): now also R21.1; no longer R12.1
- net at D3.1 (K): now also C?.1, U?.1 (IN)
- net CTL: now reaches U5.2 (GP5)
- net CTL: now also R?.2
- net at Q3.3 (B): now also R12.1; no longer R13.1
- net at Q5.3 (B): now also R13.2; no longer R21.1
- new net: D9.1 (K), Q?.1 (E)
- new net: Q?.3 (B), R?.2
- new net: Q?.2 (B), R?.1
- new net: Q?.3 (C), R?.1
- no-connect marks 1 -> 0
Other:
- note added: "Charge Control"
- moved on the sheet: BT1, C1, C10, C15, C16, C17, C18, C19, C2, C20, C21, C22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
