File: hardware-discrete/hardware-discrete.sch (KiCad schematic (older format))
At the start: 97 parts, among them J1 12V, J2 Conn_01x05, M1 5V, Q1 FQP13N06L, Q2 BD137, Q3 BD137, Q4 BD137, Q5 BD137, Q6 BD136, Q7 2N3904, SW1 F/S Mode, SW2 On/Off, U1 L7809, U2 LM7824_TO220, U3 NE555, U4 LM358, U5 L7805, U6 PIC12F675-IP, U7 LM393

Commit message: Noise source for discrete version.
Parts:
- removed JP3: MCU Isolation, Connector_PinHeader_2.54mm:PinHeader_1x02_P2.54mm_Vertical, symbol Device:Jumper_NC_Small
- removed Q6: BD136, Package_TO_SOT_THT:TO-126-3_Vertical, symbol Transistor_BJT:BD136
- removed Q7: 2N3904, Package_TO_SOT_THT:TO-92_Inline, symbol Transistor_BJT:2N3904
- removed R33: 10k, Resistor_THT:R_Axial_DIN0516_L15.5mm_D5.0mm_P5.08mm_Vertical, symbol Device:R
- removed R34: 2.2, Resistor_THT:R_Axial_DIN0516_L15.5mm_D5.0mm_P5.08mm_Vertical, symbol Device:R
- removed SW2: On/Off, symbol Switch:SW_SPST
- added C47: 1μF, Capacitor_SMD:C_0805_2012Metric_Pad1.15x1.40mm_HandSolder, symbol Device:C
- added C48, C50: 0.1μF, Capacitor_SMD:C_0805_2012Metric_Pad1.15x1.40mm_HandSolder, symbol Device:C
- added C54: 47pF, Capacitor_SMD:C_0805_2012Metric_Pad1.15x1.40mm_HandSolder, symbol Device:C
- added C55: 10μF, Capacitor_SMD:C_0805_2012Metric_Pad1.15x1.40mm_HandSolder, symbol Device:C
- added C56: 1nF, Capacitor_SMD:C_0805_2012Metric_Pad1.15x1.40mm_HandSolder, symbol Device:C
- added C58: 10μF, Capacitor_SMD:C_0805_2012Metric_Pad1.15x1.40mm_HandSolder, symbol Device:C_Small
- added C?: 1μF, Capacitor_THT:CP_Radial_D5.0mm_P2.00mm, symbol Device:CP
- added C?: 0.1μF, Capacitor_THT:CP_Radial_D5.0mm_P2.00mm, symbol Device:CP
- added D12: 10V, Diode_SMD:D_MiniMELF, symbol Device:D_Zener
- added D? (x2): 4.5V, symbol Device:D_Zener
- added D?: 1N4007, Diode_THT:D_DO-41_SOD81_P7.62mm_Horizontal, symbol Device:D
- added JP?: MCU Isolation, Connector_PinHeader_2.54mm:PinHeader_1x02_P2.54mm_Vertical, symbol Device:Jumper_NC_Small
- added Q2: MBT2222, Package_TO_SOT_SMD:SOT-23, symbol Transistor_BJT:PN2222A
- added R39: 2k, Resistor_SMD:R_0805_2012Metric_Pad1.15x1.40mm_HandSolder, symbol Device:R
- added R40: 3.3k, Resistor_SMD:R_0805_2012Metric_Pad1.15x1.40mm_HandSolder, symbol Device:R
- added R44: 27k, Resistor_SMD:R_0805_2012Metric_Pad1.15x1.40mm_HandSolder, symbol Device:R
- added R45: 6.8k, Resistor_SMD:R_0805_2012Metric_Pad1.15x1.40mm_HandSolder, symbol Device:R
- added R50: 10, Resistor_SMD:R_0805_2012Metric_Pad1.15x1.40mm_HandSolder, symbol Device:R
- added SW?: On/Off, symbol Switch:SW_SPST
- added U14: LM386, Package_SO:SO-8_5.3x6.2mm_P1.27mm, symbol Amplifier_Audio:LM386
- D7: value BLUE -> GREEN
- J2: value Conn_01x05 -> Pickit 2
- R11: value 62 -> 10k
- R13: value 1k -> 100
- R14: value 180 -> 1k
- R17: value 2.2 -> 4.7
- R18: value 15 -> 12
- R35: value 100 -> 1k; footprint Resistor_THT:R_Axial_DIN0207_L6.3mm_D2.5mm_P7.62mm_Horizontal -> Resistor_SMD:R_0805_2012Metric_Pad1.15x1.40mm_HandSolder
Connections:
- net BGND: now also D?.2 (A)
- net BREF: now also JP4.2; no longer JP4.1
- net CHG: now also R28.1, R29.2, D?.2 (A)
- net DC: now also C21.1, R13.2, U5.1 (IN), SW?.2 (B)
- net GND: now also C47.1, C48.1, C55.1, C56.1, C?.2, C?.2, D?.2 (A), JP?.1, Q2.1 (E), R40.2, R50.2, U14.2 (-), U14.4 (GND); no longer J2.5 (Pin_5), U6.8 (VSS)
- net PWR: now also C20.1; no longer C21.1
- net S2: now also U6.5 (GP2); no longer U6.2 (GP5)
- net S3: now also R10.2, U6.2 (GP5); no longer J2.2 (Pin_2), U6.4 (GP3)
- net VDD: now also J2.2 (Pin_2); no longer J2.1 (Pin_1)
- net at C17.1, C18.1, JP1.2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: now also D?.1 (K)
- net at R11.1, R14.2: now also JP4.1, C?.1, C?.1, D?.1 (K); no longer JP4.2
- net at R35.1: now also C47.2, C48.2, R40.1, U14.7 (BYPASS)
- net CTL renamed Boost
- net Boost: now also R39.1; no longer U6.5 (GP2)
- net S1 renamed CLK
- net CLK: now also J2.5 (Pin_5); no longer J2.3 (Pin_3)
- new net: D?.1 (K), SW?.1 (A)
- new net: D12.2 (A), Q2.2 (B)
- new net: Q2.3 (C), R39.2, R44.1, R45.2
- new net: C55.2, D12.1 (K), R44.2
- new net: C58.2, U14.1 (GAIN)
- new net: C50.2, U14.3 (+)
- new net: C58.1, U14.8 (GAIN)
- new net: C54.2, R50.1
- new net: C50.1, C56.2, R45.1
- new net Noise: C54.1, U14.5
- new net VPP: J2.1 (Pin_1), U6.4 (GP3)
- new net VSS: J2.3 (Pin_3), JP?.2, U6.8 (VSS)
- no-connect marks 0 -> 1
Other:
- note added: "LOAD"
- note added: "Noise Source"
- note added: "Note: Dead battery should be a battery which voltage doesn't change in a pre-determined duration of time. Use interrupt"
- note removed: "Charge Control"
- note removed: "Note: Arrangement will be altered to match the Pickit one."
- note removed: "Pickit: 1-2-5-4-3"
- moved on the sheet: BT1, C16, C17, C18, C19, C20, C21, C22, C23, C24, C25, C26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
