File: hardware-discrete/_autosave-hardware-discrete.sch (KiCad schematic (older format))
At the start: 97 parts, among them J1 12V, J2 Conn_01x05, M1 5V, Q1 FQP13N06L, Q2 BD137, Q3 BD137, Q4 BD137, Q5 BD137, Q6 BD136, Q7 2N3904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

Commit message: Minor tweaks to battery management.
Parts:
- R13: value 1k -> 100
Changed lines of the file:
@@
 P 9800 4500
 F 0 "R13" H 9730 4454 50  0000 R CNN
-F 1 "1k" H 9730 4545 50  0000 R CNN
+F 1 "100" H 9730 4545 50  0000 R CNN
 F 2 "Resistor_THT:R_Axial_DIN0516_L15.5mm_D5.0mm_P5.08mm_Vertical" V 9730 4500 50  0001 C CNN
 F 3 "~" H 9800 4500 50  0001 C CNN
