File: hardware-modular/cvco/cvco.sch (KiCad schematic (older format))
At the start: 18 parts, among them J1 SMA, U2 NLB-310-T1, Y1 CVCO55CW

Commit message: Li-Po charger module - schema.
Other:
- moved on the sheet: J?
Changed lines of the file:
@@
 L Connector_Generic:Conn_01x03 J?
 U 1 1 600AB471
-P 2700 5600
-F 0 "J?" H 2618 5917 50  0000 C CNN
-F 1 "INPUT" H 2618 5826 50  0000 C CNN
-F 2 "" H 2700 5600 50  0001 C CNN
-F 3 "~" H 2700 5600 50  0001 C CNN
-	1    2700 5600
+P 5750 1800
+F 0 "J?" H 5668 2117 50  0000 C CNN
+F 1 "INPUT" H 5668 2026 50  0000 C CNN
+F 2 "" H 5750 1800 50  0001 C CNN
+F 3 "~" H 5750 1800 50  0001 C CNN
+	1    5750 1800
 	-1   0    0    -1
 $EndComp
@@
 $EndComp
 Wire Wire Line
-	2900 5500 3050 5500
+	5950 1700 6100 1700
 Wire Wire Line
-	3050 5500 3050 5350
+	6100 1700 6100 1550
 Wire Wire Line
-	3050 5850 3050 5700
+	6100 2050 6100 1900
 Wire Wire Line
-	3050 5700 2900 5700
+	6100 1900 5950 1900
 Wire Wire Line
-	2900 5600 3200 5600
+	5950 1800 6250 1800
 $Comp
 L Regulator_Linear:LM317_TO-220 U?
@@
 	1    0    0    -1
 $EndComp
-Text GLabel 3200 5600 2    50   Input ~ 0
+Text GLabel 6250 1800 2    50   Input ~ 0
 VT
 $Comp
 L power:GND #PWR?
 U 1 1 600BCEEC
-P 3050 5850
-F 0 "#PWR?" H 3050 5600 50  0001 C CNN
-F 1 "GND" H 3055 5677 50  0000 C CNN
-F 2 "" H 3050 5850 50  0001 C CNN
-F 3 "" H 3050 5850 50  0001 C CNN
-	1    3050 5850
+P 6100 2050
+F 0 "#PWR?" H 6100 1800 50  0001 C CNN
+F 1 "GND" H 6105 1877 50  0000 C CNN
+F 2 "" H 6100 2050 50  0001 C CNN
+F 3 "" H 6100 2050 50  0001 C CNN
+	1    6100 2050
 	1    0    0    -1
 $EndComp
@@
 L power:+24V #PWR?
 U 1 1 600BE057
-P 3050 5350
-F 0 "#PWR?" H 3050 5200 50  0001 C CNN
-F 1 "+24V" H 3065 5523 50  0000 C CNN
-F 2 "" H 3050 5350 50  0001 C CNN
-F 3 "" H 3050 5350 50  0001 C CNN
-	1    3050 5350
+P 6100 1550
+F 0 "#PWR?" H 6100 1400 50  0001 C CNN
+F 1 "+24V" H 6115 1723 50  0000 C CNN
+F 2 "" H 6100 1550 50  0001 C CNN
+F 3 "" H 6100 1550 50  0001 C CNN
+	1    6100 1550
 	1    0    0    -1
 $EndComp
