File: hardware-modular/charger/charger.sch (KiCad schematic (older format))
At the start: 77 parts, among them J1 DC_IN, J2 Pickit 2, J3 BAT_OUT_4, J4 BAT_OUT_1, J5 BAT_OUT_2, J6 BAT_OUT_3, Q1 IRF9510, Q2 BD137, Q3 BD136, Q4 BD137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

Commit message: Li-Po charger module - PCB.
Parts:
- added R20: 100, Resistor_THT:R_Axial_DIN0207_L6.3mm_D2.5mm_P10.16mm_Horizontal, symbol Device:R
- J2: footprint Connector_PinHeader_2.00mm:PinHeader_1x06_P2.00mm_Vertical -> Connector_PinSocket_2.54mm:PinSocket_1x06_P2.54mm_Vertical
- R3: value 270 -> 220
- SW1: footprint Diode_THT:D_DO-41_SOD81_P10.16mm_Horizontal -> Connector_Molex:Molex_KK-254_AE-6410-02A_1x02_P2.54mm_Vertical
Connections:
- net VDD: now also C1.1, C2.1, C3.1, C4.1
- net PROBE: now reaches U2.2 (T1CKI/OSC1/CLKIN/RA5)
- net PROBE: now also R20.2
- net at BT1.1 (+), Q3.2 (C), R7.2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: now also R20.1
- new net: JP2.1, R2.1
- no-connect marks 13 -> 12
Other:
- moved on the sheet: C1, C2, C3, C4, JP2, R2
Changed lines of the file:
@@
 L Device:C C1
 U 1 1 600CEFF8
-P 7050 2050
-F 0 "C1" H 7165 2096 50  0000 L CNN
-F 1 "100nF" H 7165 2005 50  0000 L CNN
-F 2 "Capacitor_THT:C_Disc_D3.0mm_W1.6mm_P2.50mm" H 7088 1900 50  0001 C CNN
-F 3 "~" H 7050 2050 50  0001 C CNN
-	1    7050 2050
+P 7050 2250
+F 0 "C1" H 7165 2296 50  0000 L CNN
+F 1 "100nF" H 7165 2205 50  0000 L CNN
+F 2 "Capacitor_THT:C_Disc_D3.0mm_W1.6mm_P2.50mm" H 7088 2100 50  0001 C CNN
+F 3 "~" H 7050 2250 50  0001 C CNN
+	1    7050 2250
 	1    0    0    -1
 $EndComp
@@
 L Device:C C2
 U 1 1 600CF559
-P 7550 2050
-F 0 "C2" H 7665 2096 50  0000 L CNN
-F 1 "100nF" H 7665 2005 50  0000 L CNN
-F 2 "Capacitor_THT:C_Disc_D3.0mm_W1.6mm_P2.50mm" H 7588 1900 50  0001 C CNN
-F 3 "~" H 7550 2050 50  0001 C CNN
-	1    7550 2050
+P 7550 2250
+F 0 "C2" H 7665 2296 50  0000 L CNN
+F 1 "100nF" H 7665 2205 50  0000 L CNN
+F 2 "Capacitor_THT:C_Disc_D3.0mm_W1.6mm_P2.50mm" H 7588 2100 50  0001 C CNN
+F 3 "~" H 7550 2250 50  0001 C CNN
+	1    7550 2250
 	1    0    0    -1
 $EndComp
@@
 L Device:C C3
 U 1 1 600CF826
-P 8150 2050
-F 0 "C3" H 8265 2096 50  0000 L CNN
-F 1 "10nF" H 8265 2005 50  0000 L CNN
-F 2 "Capacitor_THT:C_Disc_D3.0mm_W1.6mm_P2.50mm" H 8188 1900 50  0001 C CNN
-F 3 "~" H 8150 2050 50  0001 C CNN
-	1    8150 2050
+P 8150 2250
+F 0 "C3" H 8265 2296 50  0000 L CNN
+F 1 "10nF" H 8265 2205 50  0000 L CNN
+F 2 "Capacitor_THT:C_Disc_D3.0mm_W1.6mm_P2.50mm" H 8188 2100 50  0001 C CNN
+F 3 "~" H 8150 2250 50  0001 C CNN
+	1    8150 2250
 	1    0    0    -1
 $EndComp
@@
 L Device:C C4
 U 1 1 600CFB5A
-P 8650 2050
-F 0 "C4" H 8765 2096 50  0000 L CNN
-F 1 "10nF" H 8765 2005 50  0000 L CNN
-F 2 "Capacitor_THT:C_Disc_D3.0mm_W1.6mm_P2.50mm" H 8688 1900 50  0001 C CNN
-F 3 "~" H 8650 2050 50  0001 C CNN
-	1    8650 2050
-	1    0    0    -1
-$EndComp
-Wire Wire Line
-	7050 2200 7050 2350
-Wire Wire Line
-	7050 2350 7550 2350
-Wire Wire Line
-	8650 2350 8650 2200
-Wire Wire Line
-	8150 2200 8150 2350
-Wire Wire Line
-	8150 2350 8650 2350
-Wire Wire Line
-	7550 2200 7550 2350
-Wire Wire Line
-	7550 2350 7850 2350
-Wire Wire Line
-	8650 1900 8650 1750
-Wire Wire Line
-	8650 1750 8150 1750
-Wire Wire Line
-	7050 1750 7050 1900
-Wire Wire Line
-	7550 1750 7050 1750
-Wire Wire Line
-	8150 1900 8150 1750
-Wire Wire Line
-	8150 1750 7550 1750
+P 8650 2250
+F 0 "C4" H 8765 2296 50  0000 L CNN
+F 1 "10nF" H 8765 2205 50  0000 L CNN
+F 2 "Capacitor_THT:C_Disc_D3.0mm_W1.6mm_P2.50mm" H 8688 2100 50  0001 C CNN
+F 3 "~" H 8650 2250 50  0001 C CNN
+	1    8650 2250
+	1    0    0    -1
+$EndComp
+Wire Wire Line
+	7050 2400 7050 2550
+Wire Wire Line
+	7050 2550 7550 2550
+Wire Wire Line
+	8650 2550 8650 2400
+Wire Wire Line
+	8150 2400 8150 2550
+Wire Wire Line
+	8150 2550 8650 2550
+Wire Wire Line
+	7550 2400 7550 2550
+Wire Wire Line
+	7550 2550 7850 2550
+Wire Wire Line
+	8650 2100 8650 1950
+Wire Wire Line
+	8650 1950 8150 1950
+Wire Wire Line
+	7050 1950 7050 2100
+Wire Wire Line
+	7550 1950 7050 1950
+Wire Wire Line
+	8150 2100 8150 1950
+Wire Wire Line
+	8150 1950 7550 1950
 Wire Wire Line
 	1650 2500 1650 2350
@@
 $EndComp
 Wire Wire Line
-	9000 1750 8650 1750
-Connection ~ 8650 1750
-Wire Wire Line
-	9000 1750 9000 2450
-Wire Wire Line
-	7850 2350 7850 2500
-Wire Wire Line
-	7850 2350 8150 2350
+	9000 1950 8650 1950
+Connection ~ 8650 1950
+Wire Wire Line
+	7850 2550 7850 2700
+Wire Wire Line
+	7850 2550 8150 2550
 $Comp
 L power:GND #PWR04
 U 1 1 600DDA9E
-P 7850 2500
-F 0 "#PWR04" H 7850 2250 50  0001 C CNN
-F 1 "GND" H 7855 2327 50  0000 C CNN
-F 2 "" H 7850 2500 50  0001 C CNN
-F 3 "" H 7850 2500 50  0001 C CNN
-	1    7850 2500
-	1    0    0    -1
-$EndComp
-Wire Wire Line
-	7550 1900 7550 1750
+P 7850 2700
+F 0 "#PWR04" H 7850 2450 50  0001 C CNN
+F 1 "GND" H 7855 2527 50  0000 C CNN
+F 2 "" H 7850 2700 50  0001 C CNN
+F 3 "" H 7850 2700 50  0001 C CNN
+	1    7850 2700
+	1    0    0    -1
+$EndComp
+Wire Wire Line
+	7550 2100 7550 1950
 Wire Wire Line
 	9000 4700 9000 4850
@@
 L Device:R R2
 U 1 1 600E9D04
-P 6750 1750
-F 0 "R2" V 6543 1750 50  0000 C CNN
-F 1 "22" V 6634 1750 50  0000 C CNN
-F 2 "Resistor_THT:R_Axial_DIN0414_L11.9mm_D4.5mm_P5.08mm_Vertical" V 6680 1750 50  0001 C CNN
-F 3 "~" H 6750 1750 50  0001 C CNN
-	1    6750 1750
+P 6400 1950
+F 0 "R2" V 6193 1950 50  0000 C CNN
+F 1 "22" V 6284 1950 50  0000 C CNN
+F 2 "Resistor_THT:R_Axial_DIN0414_L11.9mm_D4.5mm_P5.08mm_Vertical" V 6330 1950 50  0001 C CNN
+F 3 "~" H 6400 1950 50  0001 C CNN
+	1    6400 1950
 	0    1    1    0
 $EndComp
 Wire Wire Line
-	7050 1750 6900 1750
-Connection ~ 7050 1750
-Connection ~ 7550 2350
-Connection ~ 7550 1750
-Connection ~ 7850 2350
-Connection ~ 8150 2350
-Connection ~ 8150 1750
+	6700 1950 6550 1950
+Connection ~ 7550 2550
+Connection ~ 7550 1950
+Connection ~ 7850 2550
+Connection ~ 8150 2550
+Connection ~ 8150 1950
 Wire Wire Line
 	10500 3550 10650 3550
 Text GLabel 10650 3550 2    50   Input ~ 0
 VPP
-Text GLabel 9150 2800 2    50   Input ~ 0
+Text GLabel 7050 1800 1    50   Input ~ 0
 VDD
 Text GLabel 9150 4700 2    50   Input ~ 0
@@
 L Device:Jumper_NC_Small JP2
 U 1 1 600FF35F
-P 9000 2550
-F 0 "JP2" V 8954 2625 50  0000 L CNN
-F 1 "Jumper" V 9045 2625 50  0000 L CNN
-F 2 "Connector_PinHeader_2.54mm:PinHeader_1x02_P2.54mm_Vertical" H 9000 2550 50  0001 C CNN
-F 3 "~" H 9000 2550 50  0001 C CNN
-	1    9000 2550
-	0    1    1    0
-$EndComp
-Wire Wire Line
-	9000 2650 9000 2800
-Wire Wire Line
-	9000 2800 9150 2800
-Wire Wire Line
-	9000 2800 9000 2950
-Connection ~ 9000 2800
+P 6800 1950
+F 0 "JP2" H 6800 2162 50  0000 C CNN
+F 1 "Jumper" H 6800 2071 50  0000 C CNN
+F 2 "Connector_PinHeader_2.54mm:PinHeader_1x02_P2.54mm_Vertical" H 6800 1950 50  0001 C CNN
+F 3 "~" H 6800 1950 50  0001 C CNN
+	1    6800 1950
+	1    0    0    -1
+$EndComp
+Wire Wire Line
+	7050 1950 7050 1800
 $Comp
 L Device:Jumper_NC_Small JP3
@@
 Text GLabel 10650 3950 2    50   Input ~ 0
 PWM
-NoConn ~ 10500 3750
 NoConn ~ 10500 4050
 NoConn ~ 10500 4150
@@
 F 0 "J2" V 6772 4662 50  0000 R CNN
 F 1 "Pickit 2" V 6863 4662 50  0000 R CNN
-F 2 "Connector_PinHeader_2.00mm:PinHeader_1x06_P2.00mm_Vertical" H 6900 5050 50  0001 C CNN
+F 2 "Connector_PinSocket_2.54mm:PinSocket_1x06_P2.54mm_Vertical" H 6900 5050 50  0001 C CNN
 F 3 "~" H 6900 5050 50  0001 C CNN
 	1    6900 5050
@@
 F 0 "SW1" H 3750 7585 50  0000 C CNN
 F 1 "ON/OFF" H 3750 7494 50  0000 C CNN
-F 2 "Diode_THT:D_DO-41_SOD81_P10.16mm_Horizontal" H 3750 7350 50  0001 C CNN
+F 2 "Connector_Molex:Molex_KK-254_AE-6410-02A_1x02_P2.54mm_Vertical" H 3750 7350 50  0001 C CNN
 F 3 "~" H 3750 7350 50  0001 C CNN
 	1    3750 7350
@@
 Optional Regulator
 Wire Wire Line
-	6600 1750 6450 1750
-Text GLabel 6450 1750 0    50   Input ~ 0
+	6250 1950 6100 1950
+Text GLabel 6100 1950 0    50   Input ~ 0
 DC
 Wire Notes Line
 	11050 5550 11050 1400
 Wire Notes Line
-	11050 1400 6150 1400
-Wire Notes Line
-	6150 1400 6150 5550
-Wire Notes Line
-	6150 5550 11050 5550
+	11050 1400 5800 1400
+Wire Notes Line
+	5800 1400 5800 5550
+Wire Notes Line
+	5800 5550 11050 5550
 Text Notes 10150 1600 0    50   ~ 0
 Battery Management
@@
 P 14650 2900
 F 0 "R3" V 14443 2900 50  0000 C CNN
-F 1 "270" V 14534 2900 50  0000 C CNN
+F 1 "220" V 14534 2900 50  0000 C CNN
 F 2 "Resistor_THT:R_Axial_DIN0207_L6.3mm_D2.5mm_P10.16mm_Horizontal" V 14580 2900 50  0001 C CNN
 F 3 "~" H 14650 2900 50  0001 C CNN
@@
 Wire Wire Line
 	3700 6000 3850 6000
-Wire Wire Line
-	3400 6200 3400 7350
 $Comp
 L power:GND #PWR0101
@@
 Wire Wire Line
 	4450 5900 4600 5900
+Entry Wire Line
+	-650 6250 -550 6350
+Wire Wire Line
+	9000 1950 9000 2950
+Wire Wire Line
+	6900 1950 7050 1950
+Connection ~ 7050 1950
+Wire Wire Line
+	3400 6750 3250 6750
+Text GLabel 2800 6750 0    50   Input ~ 0
+PROBE
+Wire Wire Line
+	10500 3750 10650 3750
+Text GLabel 10650 3750 2    50   Input ~ 0
+PROBE
+Connection ~ 3400 6750
+Wire Wire Line
+	3400 6750 3400 7350
+Wire Wire Line
+	3400 6200 3400 6750
+$Comp
+L Device:R R20
+U 1 1 602609AB
+P 3100 6750
+F 0 "R20" V 2893 6750 50  0000 C CNN
+F 1 "100" V 2984 6750 50  0000 C CNN
+F 2 "Resistor_THT:R_Axial_DIN0207_L6.3mm_D2.5mm_P10.16mm_Horizontal" V 3030 6750 50  0001 C CNN
+F 3 "~" H 3100 6750 50  0001 C CNN
+	1    3100 6750
+	0    1    1    0
+$EndComp
+Wire Wire Line
+	2950 6750 2800 6750
 $EndSCHEMATC

Commit message: Gerber files - Charger.
Connections:
- net SWITCH: no longer names the net of U2.15 (RC1/AN5/C12IN1-)
- no-connect marks 12 -> 13
Changed lines of the file:
@@
 Battery Management
-Wire Wire Line
-	7500 3350 7350 3350
-Text GLabel 7350 3350 0    50   Input ~ 0
-SWITCH
 Wire Wire Line
 	3650 3400 3650 3500
@@
 Wire Wire Line
 	2950 6750 2800 6750
+NoConn ~ 7500 3350
 $EndSCHEMATC
