File: hardware-modular/amplifiers/adl-variant/adl-variant.kicad_pcb (KiCad board)
At the start: 2 copper layers, 60 x 40 mm, 20 parts, among them J1 DC_IN, J2 RF_IN, J3 RF_OUT, U1 ADL5602

Commit message: Tweaked amplifier modules.
Other:
- board text added: "IN"
- board text added: "OUT"

Commit message: Trans. line width issue resolved - amp. modules.
Routing:
- net Net-(C7-Pad2): track 7.05 -> 7.55 mm
Changed lines of the file:
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@@
   (general
     (thickness 1.6)
-    (drawings 19)
-    (tracks 7)
+    (drawings 20)
+    (tracks 8)
     (zones 0)
     (modules 20)
@@
   )
   (setup
-    (last_trace_width 0.25)
+    (last_trace_width 0.784566)
     (user_trace_width 0.525491)
-    (user_trace_width 1.04516)
+    (user_trace_width 0.784566)
     (trace_clearance 0.2)
-    (zone_clearance 0.2)
+    (zone_clearance 0.15)
     (zone_45_only no)
     (trace_min 0.2)
@@
     (visible_elements 7FFFFF7F)
     (pcbplotparams
-      (layerselection 0x010fc_ffffffff)
+      (layerselection 0x010f0_ffffffff)
       (usegerberextensions false)
       (usegerberattributes true)
       (usegerberadvancedattributes true)
       (creategerberjobfile true)
-      (excludeedgelayer true)
+      (excludeedgelayer false)
       (linewidth 0.100000)
       (plotframeref false)
@@
       (outputformat 1)
       (mirror false)
-      (drillshape 1)
+      (drillshape 0)
       (scaleselection 1)
-      (outputdirectory ""))
+      (outputdirectory "gerber/"))
   )
   (net 0 "")
@@
       (net 2 GND))
   )
+  (gr_line (start 139.05 66.5) (end 135.4 66.5) (layer F.Mask) (width 1.084566))
+  (gr_line (start 131.5 66.5) (end 135.4 66.5) (layer F.Mask) (width 1.084566))
+  (gr_line (start 140.95 66.5) (end 157 66.5) (layer F.Mask) (width 1.084566))
+  (gr_line (start 120.95 66.5) (end 128.5 66.5) (layer F.Mask) (width 1.084566))
+  (gr_line (start 103 66.5) (end 119.05 66.5) (layer F.Mask) (width 1.084566))
   (gr_text OUT (at 157 73) (layer F.SilkS)
     (effects (font (size 1 1) (thickness 0.12)))
@@
     (effects (font (size 1 1) (thickness 0.12)))
   )
-  (gr_line (start 140.95 66.5) (end 157 66.5) (layer F.Mask) (width 1.44516))
-  (gr_line (start 131.5 66.5) (end 139.05 66.5) (layer F.Mask) (width 1.44516))
-  (gr_line (start 120.95 66.5) (end 128 66.5) (layer F.Mask) (width 1.44516))
-  (gr_line (start 119.05 66.5) (end 103 66.5) (layer F.Mask) (width 1.44516))
   (dimension 60 (width 0.15) (layer Dwgs.User)
     (gr_text "60.000 mm" (at 130 43.7) (layer Dwgs.User)
@@
   (segment (start 137 84) (end 135.4 82.4) (width 0.525491) (layer F.Cu) (net 1))
   (segment (start 142.5 84) (end 137 84) (width 0.525491) (layer F.Cu) (net 1))
-  (segment (start 119.05 66.5) (end 103 66.5) (width 1.04516) (layer F.Cu) (net 3))
-  (segment (start 120.95 66.5) (end 128 66.5) (width 1.04516) (layer F.Cu) (net 4))
-  (segment (start 140.95 66.5) (end 157 66.5) (width 1.04516) (layer F.Cu) (net 5))
-  (segment (start 131.5 66.5) (end 139.05 66.5) (width 1.04516) (layer F.Cu) (net 6))
+  (segment (start 103 66.5) (end 119.05 66.5) (width 0.784566) (layer F.Cu) (net 3))
+  (segment (start 120.95 66.5) (end 128.5 66.5) (width 0.784566) (layer F.Cu) (net 4))
+  (segment (start 140.95 66.5) (end 157 66.5) (width 0.784566) (layer F.Cu) (net 5))
+  (segment (start 131.5 66.5) (end 135.4 66.5) (width 0.784566) (layer F.Cu) (net 6))
+  (segment (start 139.05 66.5) (end 135.4 66.5) (width 0.784566) (layer F.Cu) (net 6))
   (zone (net 2) (net_name GND) (layer F.Cu) (hatch edge 0.508)
-    (connect_pads yes (clearance 0.2))
-    (min_thickness 0.1)
-    (fill yes (arc_segments 32) (thermal_gap 0.2) (thermal_bridge_width 0.2))
+    (connect_pads yes (clearance 0.15))
+    (min_thickness 0.075)
+    (fill yes (arc_segments 32) (thermal_gap 0.15) (thermal_bridge_width 0.15))
     (polygon
       (pts
@@
   )
   (zone (net 2) (net_name GND) (layer B.Cu) (hatch edge 0.508)
-    (connect_pads yes (clearance 0.2))
-    (min_thickness 0.1)
-    (fill yes (arc_segments 32) (thermal_gap 0.2) (thermal_bridge_width 0.2))
+    (connect_pads yes (clearance 0.15))
+    (min_thickness 0.075)
+    (fill yes (arc_segments 32) (thermal_gap 0.15) (thermal_bridge_width 0.15))
     (polygon
       (pts
