File: hardware-modular/vco-variants/500-1000-cvco/500-1000-cvco.sch (KiCad schematic (older format))
At the start: 29 parts

Commit message: CVCO 500-1000 MHz module - PCB.
Parts:
- C1: renamed from C?; footprint (none) -> Capacitor_THT:C_Disc_D3.0mm_W1.6mm_P2.50mm
- C10, C2, C3, C4, C5, C6, C7, C8, C9: renamed from C?; footprint (none) -> Capacitor_SMD:C_0805_2012Metric
- D1, D2, D3, D4, D5: renamed from D?; footprint (none) -> Diode_THT:D_DO-41_SOD81_P2.54mm_Vertical_AnodeUp
- H1, H2, H3, H4: renamed from H?; footprint (none) -> MountingHole:MountingHole_3.2mm_M3_Pad_Via
- J1: renamed from J?; footprint (none) -> TerminalBlock_4Ucon:TerminalBlock_4Ucon_1x03_P3.50mm_Vertical
- J2: renamed from J?; footprint (none) -> Connector_Coaxial:SMA_Amphenol_132289_EdgeMount
- JP1: renamed from JP?; footprint (none) -> Connector_PinHeader_2.54mm:PinHeader_1x02_P2.54mm_Vertical
- L1: renamed from L?; footprint (none) -> Inductor_SMD:L_0805_2012Metric
- R1: renamed from R?; footprint (none) -> Resistor_THT:R_Axial_DIN0309_L9.0mm_D3.2mm_P15.24mm_Horizontal
- R2, R3, R4, R5: renamed from R?; footprint (none) -> Resistor_THT:R_Axial_DIN0207_L6.3mm_D2.5mm_P10.16mm_Horizontal
- gave numbers to parts that had none: 1
Connections:
- net GND: now also JP1.1; no longer C10.2, C9.2
- net at D2.1 (K), D5.1 (K), R5.1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: now also C10.1, C9.1; no longer JP1.1
- new net: C10.2, C9.2, JP1.2
Other:
- moved on the sheet: C10, C9, JP1
