File: hardware-modular/psu/psu.kicad_pcb (KiCad board)
At the start: 2 copper layers, 95 x 60 mm, 52 parts, among them J1 DC_OUT_1, J2 DC_OUT_2, J3 DC_OUT_3, J4 DC_OUT_4, J5 DC_IN, Q1 BD137, Q2 BD137, Q3 BD137, Q4 BD137, Q5 IRF9510, U1 L7805

Commit message: PSU module revision.
Parts:
- removed the G*** at (129.3, 64.9)
- R1: value 100 -> 2.2; footprint Resistor_THT:R_Axial_DIN0207_L6.3mm_D2.5mm_P10.16mm_Horizontal -> Resistor_THT:R_Axial_DIN0309_L9.0mm_D3.2mm_P12.70mm_Horizontal
- R6: footprint Resistor_THT:R_Axial_DIN0207_L6.3mm_D2.5mm_P10.16mm_Horizontal -> Resistor_THT:R_Axial_DIN0309_L9.0mm_D3.2mm_P12.70mm_Horizontal
- moved D9 12.0 mm to (140.0, 84.4)
- moved R1 10.2 mm to (112.6, 102.0), turned to 0 degrees
- moved C1 5.00 mm to (148.0, 58.9)
- moved C2 5.00 mm to (148.0, 73.0)
- moved C3 5.00 mm to (148.0, 87.0)
- moved C4 5.00 mm to (148.0, 101.2)
- moved C5 5.00 mm to (127.5, 84.5)
- moved C6 5.00 mm to (127.5, 94.5)
- moved D11 5.00 mm to (141.1, 61.5)
- moved F1 5.00 mm to (162.2, 63.3)
- moved H2 5.00 mm to (164.0, 56.0)
- moved H3 5.00 mm to (164.0, 104.0)
- moved HS1 5.00 mm to (136.0, 89.5)
- moved J5 5.00 mm to (163.0, 95.9)
- moved Q5 5.00 mm to (133.5, 56.5)
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Connections:
- JP5 pad 1: Net-(JP5-Pad1) -> GND
- JP5 pad 2: Net-(J1-Pad1) -> Net-(JP5-Pad2)
- R1 pad 1: Net-(JP5-Pad1) -> Net-(Q1-Pad1)
- R1 pad 2: Net-(D1-Pad2) -> Net-(JP5-Pad2)
Routing:
- net Net-(Q1-Pad1): track 4.29 -> 20.4 mm
- net Net-(J1-Pad1): track 68.9 -> 56.3 mm
- net Net-(JP5-Pad2): track 0.00 -> 11.1 mm
- net Net-(C1-Pad1): track 90.8 -> 101.0 mm
- net Net-(JP5-Pad1): track 9.07 -> 0.00 mm
- net Net-(D1-Pad2): track 25.2 -> 22.9 mm
- net Net-(D10-Pad1): track 4.85 -> 3.76 mm
Other:
- board size 95 x 60 mm -> 90 x 60 mm
- board text added: "REV: 1.0.1"
- board text removed: "REV: 1.0.0"

Commit message: PSU module revision.
Parts:
- removed the C5 at (127.5, 84.5)
- removed D11: 18V, Diode_THT:D_DO-41_SOD81_P10.16mm_Horizontal
- removed the D2 at (108.8, 82.4)
- removed the G*** at (120.5, 56.0)
- removed Q5: IRF9510, Package_TO_SOT_THT:TO-220-3_Vertical
- removed the R1 at (112.6, 102.0)
- removed the R10 at (141.1, 66.5)
- added C1: 1mF, Capacitor_THT:CP_Radial_D10.0mm_P5.00mm, F.Cu at (149.0, 103.5)
- added C10: 1mF, Capacitor_THT:CP_Radial_D8.0mm_P3.50mm, F.Cu at (96.6, 83.3)
- added C11: 1mF, Capacitor_THT:CP_Radial_D8.0mm_P3.50mm, F.Cu at (96.6, 73.4)
- added C12: 1mF, Capacitor_THT:CP_Radial_D8.0mm_P3.50mm, F.Cu at (96.6, 63.4)
- added C7: 0.1µF, Capacitor_THT:C_Disc_D3.0mm_W1.6mm_P2.50mm, F.Cu at (130.0, 72.5)
- added C8: 100µF, Capacitor_THT:CP_Radial_D5.0mm_P2.00mm, F.Cu at (102.0, 54.5)
- added C9: 1mF, Capacitor_THT:CP_Radial_D8.0mm_P3.50mm, F.Cu at (96.6, 93.3)
- added D10: 1N4007, Diode_THT:D_DO-41_SOD81_P2.54mm_Vertical_AnodeUp, F.Cu at (122.5, 57.6)
- added G***: Lightning, Icons:Lightning, F.Cu at (158.0, 65.1)
- added L1: 100µF, Inductor_THT:L_Toroid_Vertical_L16.0mm_W8.0mm_P7.62mm, F.Cu at (137.1, 98.5)
- added R7: 2.2, Resistor_THT:R_Axial_DIN0309_L9.0mm_D3.2mm_P12.70mm_Horizontal, F.Cu at (112.3, 101.8)
- C6: value 0.1µF -> 0.33µF
- D3, D4, D5, D6, D7, D8, D9: footprint Diode_THT:D_DO-41_SOD81_P10.16mm_Horizontal -> Diode_THT:D_DO-41_SOD81_P2.54mm_Vertical_AnodeUp
- moved C5 44.7 mm to (149.0, 56.5)
- moved F1 33.4 mm to (163.0, 96.7), turned to 90 degrees
- moved C2 32.9 mm to (149.0, 91.8)
- moved J1 29.1 mm to (163.0, 66.8)
- moved D4 28.5 mm to (122.5, 87.5), turned to 0 degrees
- moved C6 27.2 mm to (130.0, 67.5)
- moved D9 26.6 mm to (125.0, 62.5), turned to 180 degrees
- moved D3 25.7 mm to (125.0, 92.4)
- moved D1 25.5 mm to (131.8, 103.5), turned to 0 degrees
- moved HS1 19.6 mm to (137.9, 70.0)
- moved U1 19.6 mm to (133.0, 67.5)
- moved C4 18.8 mm to (149.0, 68.2)
- moved R6 13.7 mm to (125.0, 97.5)
- moved D2 12.0 mm to (94.0, 55.5)
- moved Q1 10.5 mm to (104.5, 97.5)
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- renumbered C1 to C2, C2 to C3, C3 to C4, C4 to C5, D10 to D2, J5 to J1, J1 to J2, J2 to J3, J3 to J4, J4 to J5, R11 to R1, R9 to R10, R7 to R8, R8 to R9
Connections:
- net +7.5V renamed +12V
- C6 pad 1: OUT -> Net-(C1-Pad1)
- D2 pad 1: Net-(D10-Pad1) -> GND
- D2 pad 2: OUT -> Net-(C8-Pad1)
- D4 pad 1: Net-(D4-Pad1) -> GND
- D4 pad 2: Net-(D4-Pad2) -> Net-(D3-Pad1)
- D5 pad 1: GND -> Net-(D5-Pad1)
- D5 pad 2: Net-(D1-Pad1) -> Net-(D5-Pad2)
- D6 pad 2: Net-(D2-Pad1) -> Net-(D5-Pad1)
- D7 pad 1: GND -> Net-(D7-Pad1)
- D7 pad 2: Net-(D3-Pad1) -> Net-(D7-Pad2)
- D8 pad 2: Net-(D4-Pad1) -> Net-(D7-Pad1)
- D9 pad 1: Net-(C1-Pad1) -> Net-(D10-Pad2)
- D9 pad 2: OUT -> Net-(D9-Pad2)
- F1 pad 1: Net-(F1-Pad1) -> Net-(D1-Pad2)
- Q1 pad 3: Net-(D1-Pad2) -> Net-(D3-Pad2)
- Q2 pad 3: Net-(D2-Pad2) -> Net-(D5-Pad2)
- Q3 pad 3: Net-(D3-Pad2) -> Net-(D7-Pad2)
- Q4 pad 3: Net-(D4-Pad2) -> Net-(D9-Pad2)
- R1 pad 1: Net-(D10-Pad1) -> Net-(C8-Pad1)
- R1 pad 2: GND -> OUT
- R2 pad 2: Net-(D1-Pad2) -> Net-(D3-Pad2)
- R3 pad 2: Net-(D2-Pad2) -> Net-(D5-Pad2)
- R4 pad 2: Net-(D3-Pad2) -> Net-(D7-Pad2)
- R5 pad 2: Net-(D4-Pad2) -> Net-(D9-Pad2)
Routing:
- net Net-(C1-Pad1): track 101.0 -> 0.00 mm
- net Net-(F1-Pad1): track 33.8 -> 0.00 mm
- net Net-(D1-Pad2): track 22.9 -> 0.00 mm
- net Net-(C10-Pad1): track 79.3 -> 56.8 mm
- net Net-(D2-Pad2): track 20.7 -> 0.00 mm
- net Net-(D4-Pad2): track 20.7 -> 0.00 mm
- net Net-(C11-Pad1): track 88.7 -> 68.0 mm
- net Net-(D5-Pad2): track 0.00 -> 20.1 mm
- net Net-(D9-Pad2): track 0.00 -> 20.1 mm
- net Net-(D7-Pad2): track 0.00 -> 20.1 mm
- net Net-(C12-Pad1): track 100.4 -> 80.7 mm
- net +12V: track 13.3 -> 0.00 mm
- net Net-(Q5-Pad1): track 13.2 -> 0.00 mm
- net Net-(C9-Pad2): track 7.72 -> 20.1 mm
- net Net-(C10-Pad2): track 7.72 -> 19.3 mm
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- added copper zone on F.Cu, net +12V
- added copper zone on F.Cu, net Net-(C1-Pad1)
- added copper zone on F.Cu, net Net-(D1-Pad1)
- added copper zone on F.Cu, net Net-(D1-Pad2)
Other:
- board text added: "REV: 1.1.0"
- board text removed: "REV: 1.0.1"
